File: KiCad FIles/TMSHB_UART_ALL_V2/TMSHB_UART_ALL_V2.kicad_pcb (KiCad board)
At the start: 2 copper layers, 320 x 332.7 mm, 93 parts, among them J1 Conn_01x08_Pin, J10 Conn_01x02_Pin, J11 Conn_01x02_Pin, J12 Conn_01x02_Pin, J13 Conn_01x02_Pin, J14 Conn_01x02_Pin, J15 Conn_01x16_Pin, J16 Conn_01x08_Pin, J17 Conn_01x05_Pin, J18 Conn_01x05_Pin, J19 Conn_01x05_Pin, J2 Conn_01x15_Pin, J20 Conn_01x15_Pin, J21 Conn_01x15_Pin, J22 Conn_01x16_Pin, J23 Conn_01x08_Pin, J24 Conn_01x05_Pin, J25 Conn_01x05_Pin, J26 Conn_01x05_Pin, J27 Conn_01x12_Pin, J28 Conn_01x12_Pin, J29 Conn_01x12_Pin, J3 Conn_01x16_Pin, J30 Conn_01x02_Pin, J4 Conn_01x05_Pin, J5 Conn_01x05_Pin, J6 Conn_01x03_Pin, J7 Conn_01x05_Pin, J8 Conn_01x03_Pin, J9 Conn_01x02_Pin, Q10 NPN, Q11 NPN, Q12 NPN, Q13 NPN, Q14 PNP, Q2 PNP, Q3 NPN, Q8 NPN, Q9 NPN, U1 TR1602, U10 NE555P, U11 74LS138, U12 74LS32, U2 27C16, U3 74LS00, U5 NE555P, U7 TR1602, U8 74LS00, U9 74LS32

Commit message: 2026/1/13
Parts:
- removed U12: 74LS32, Package_DIP:DIP-14_W7.62mm
- added C12: C, Capacitor_THT:C_Disc_D3.0mm_W1.6mm_P2.50mm, F.Cu at (124.5, 116.8)
- added C14: C, Capacitor_THT:C_Disc_D3.0mm_W1.6mm_P2.50mm, F.Cu at (256.5, 167.6)
- added C19: 1u, Capacitor_THT:C_Disc_D3.0mm_W1.6mm_P2.50mm, F.Cu at (157.5, 88.9)
- added D11: D_Schottky, Diode_THT:D_DO-34_SOD68_P7.62mm_Horizontal, F.Cu at (144.8, 192.4)
- added D12: D_Schottky, Diode_THT:D_DO-34_SOD68_P7.62mm_Horizontal, F.Cu at (144.8, 195.6)
- added D3: D, Diode_THT:D_DO-34_SOD68_P7.62mm_Horizontal, F.Cu at (134.6, 68.6)
- added J31: Conn_01x04_Pin, Connector_PinHeader_2.54mm:PinHeader_1x04_P2.54mm_Vertical, F.Cu at (228.6, 236.2)
- added J32: Conn_01x02_Pin, Connector_PinHeader_2.54mm:PinHeader_1x02_P2.54mm_Vertical, F.Cu at (165.1, 55.9)
- added Q1: NPN, Package_TO_SOT_THT:TO-92_Inline_Wide, F.Cu at (154.9, 61.0)
- added R1: 4.7k, Resistor_THT:R_Axial_DIN0207_L6.3mm_D2.5mm_P10.16mm_Horizontal, F.Cu at (170.2, 61.0)
- added R2: 1k, Resistor_THT:R_Axial_DIN0207_L6.3mm_D2.5mm_P10.16mm_Horizontal, F.Cu at (144.8, 66.0)
- added R5: 10k, Resistor_THT:R_Axial_DIN0207_L6.3mm_D2.5mm_P10.16mm_Horizontal, F.Cu at (157.5, 78.7)
- added R8: 1k, Resistor_THT:R_Axial_DIN0207_L6.3mm_D2.5mm_P10.16mm_Horizontal, F.Cu at (144.8, 188.8)
- added U13: 74LS138, Package_DIP:DIP-16_W7.62mm, F.Cu at (137.0, 208.3)
- added U4: 74LS32, Package_DIP:DIP-14_W7.62mm, F.Cu at (129.5, 91.4)
- added U6: 74LS00, Package_DIP:DIP-14_W7.62mm, F.Cu at (129.5, 124.5)
- J27, J28, J29: footprint Connector_PinSocket_2.54mm:PinSocket_1x12_P2.54mm_Vertical -> Connector_PinHeader_2.54mm:PinHeader_1x12_P2.54mm_Vertical
- U2: value 27C16 -> 74LS04; footprint Package_DIP:DIP-24_W15.24mm -> Package_DIP:DIP-14_W7.62mm
- moved J28 303.6 mm to (101.6, 73.7)
- moved C3 195.8 mm to (132.1, 58.4)
- moved J14 170.3 mm to (193.0, 355.6)
- moved J17 170.3 mm to (185.4, 368.3)
- moved Q9 170.3 mm to (185.4, 363.2)
- moved C10 170.3 mm to (198.1, 299.8)
- moved C18 170.3 mm to (175.3, 294.6)
- moved C7 170.3 mm to (154.9, 297.1)
- moved C9 170.3 mm to (139.7, 304.8)
- moved D2 170.3 mm to (124.5, 299.7)
- moved J12 170.3 mm to (182.9, 355.6)
- moved J2 170.3 mm to (127.0, 368.3)
- moved J3 170.3 mm to (198.1, 368.3)
- moved J7 170.3 mm to (114.3, 368.3)
- moved Q10 170.3 mm to (190.5, 363.2)
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Connections:
- C17 pad 1: -12V -> Net-(J32-Pin_1)
- J27 pad 1: THRE1 -> Net-(J27-Pin_1)
- J27 pad 10: unconnected-(J27-Pin_10-Pad10) -> Net-(J27-Pin_10)
- J27 pad 11: unconnected-(J27-Pin_11-Pad11) -> Net-(J27-Pin_11)
- J27 pad 12: unconnected-(J27-Pin_12-Pad12) -> Net-(J27-Pin_12)
- J27 pad 2: /THRL1 -> Net-(J27-Pin_2)
- J27 pad 3: RRD1 -> Net-(J27-Pin_3)
- J27 pad 4: /DRR1 -> Net-(J27-Pin_4)
- J27 pad 5: unconnected-(J27-Pin_5-Pad5) -> Net-(J27-Pin_5)
- J27 pad 6: unconnected-(J27-Pin_6-Pad6) -> Net-(J27-Pin_6)
- J27 pad 7: unconnected-(J27-Pin_7-Pad7) -> Net-(J27-Pin_7)
- J27 pad 8: unconnected-(J27-Pin_8-Pad8) -> Net-(J27-Pin_8)
- J27 pad 9: unconnected-(J27-Pin_9-Pad9) -> Net-(J27-Pin_9)
- J28 pad 1: unconnected-(J28-Pin_1-Pad1) -> M0DATR
- J28 pad 2: unconnected-(J28-Pin_2-Pad2) -> M0RERD
- J28 pad 3: unconnected-(J28-Pin_3-Pad3) -> M0THRE
- J28 pad 4: unconnected-(J28-Pin_4-Pad4) -> /M0THL
- J28 pad 5: THRE2 -> /M0IQR
- J28 pad 6: /THRL2 -> unconnected-(J28-Pin_6-Pad6)
- J28 pad 7: RRD2 -> unconnected-(J28-Pin_7-Pad7)
- J28 pad 8: /DRR2 -> unconnected-(J28-Pin_8-Pad8)
- J29 pad 1: Net-(J29-Pin_1) -> unconnected-(J29-Pin_1-Pad1)
- J29 pad 10: unconnected-(J29-Pin_10-Pad10) -> /M1IQR
- J29 pad 2: Net-(J29-Pin_2) -> unconnected-(J29-Pin_2-Pad2)
- J29 pad 3: Net-(J29-Pin_3) -> unconnected-(J29-Pin_3-Pad3)
- J29 pad 4: Net-(J29-Pin_4) -> unconnected-(J29-Pin_4-Pad4)
- J29 pad 5: Net-(J29-Pin_5) -> unconnected-(J29-Pin_5-Pad5)
- J29 pad 6: Net-(J29-Pin_6) -> M1DATR
- J29 pad 7: Net-(J29-Pin_7) -> M1RERD
- J29 pad 8: Net-(J29-Pin_8) -> M1THRE
- J29 pad 9: unconnected-(J29-Pin_9-Pad9) -> /M1THL
- U1 pad 18: /DRR1 -> /M0IQR
- U1 pad 2: -12V -> Net-(J32-Pin_1)
- U1 pad 23: /THRL1 -> /M0THL
- U1 pad 4: RRD1 -> M0RERD
- U11 pad 1: Net-(U11-A0) -> AD1_3
- U11 pad 10: Net-(J29-Pin_6) -> Net-(U11-O5)
- U11 pad 11: Net-(U11-O4) -> Net-(J27-Pin_5)
- U11 pad 12: Net-(J29-Pin_4) -> Net-(J27-Pin_4)
- U11 pad 13: Net-(J29-Pin_3) -> Net-(U11-O2)
- U11 pad 14: Net-(J29-Pin_2) -> Net-(U11-O1)
- U11 pad 2: Net-(U11-A1) -> AD2_3
- U11 pad 3: Net-(U11-A2) -> AD3_3
- U11 pad 4: Net-(U11-E1) -> Net-(D11-K)
- U11 pad 5: Net-(U11-E1) -> AD4_3
- U11 pad 7: Net-(J29-Pin_8) -> Net-(U11-O7)
- U11 pad 9: Net-(J29-Pin_7) -> Net-(U11-O6)
- U2 pad 1: AD8_3 -> Net-(U11-O0)
- U2 pad 10: Net-(U11-A1) -> Net-(J27-Pin_7)
- U2 pad 11: Net-(U11-A2) -> Net-(U11-O6)
- U2 pad 12: GND -> Net-(J27-Pin_8)
- U2 pad 13: unconnected-(U2-D3-Pad13) -> Net-(U11-O7)
- U2 pad 14: unconnected-(U2-D4-Pad14) -> +5V
- U2 pad 2: AD7_3 -> Net-(J27-Pin_1)
- U2 pad 3: AD6_3 -> Net-(U11-O1)
- U2 pad 4: AD5_3 -> Net-(J27-Pin_2)
- U2 pad 5: AD4_3 -> Net-(U11-O2)
- U2 pad 6: AD3_3 -> Net-(J27-Pin_3)
- U2 pad 7: AD2_3 -> GND
- U2 pad 8: AD1_3 -> Net-(J27-Pin_6)
- U2 pad 9: Net-(U11-A0) -> Net-(U11-O5)
- U3 pad 10: Net-(U11-O0) -> AD4_3
- U3 pad 11: Net-(J29-Pin_5) -> unconnected-(U3-Pad11)
- U3 pad 12: Net-(U11-O4) -> GND
- U3 pad 13: Net-(U11-O4) -> GND
- U3 pad 8: Net-(J29-Pin_1) -> Net-(U13-E2)
- U3 pad 9: Net-(U11-O0) -> AD4_3
Routing:
- net +5V: track 624.1 -> 825.1 mm, vias 20 -> 26
- net /M0THL: track 0.00 -> 173.3 mm, vias 0 -> 3
- net Net-(J29-Pin_8): track 139.1 -> 0.00 mm, vias 3 -> 0
- net /M0IQR: track 0.00 -> 121.0 mm, vias 0 -> 4
- net Net-(U1-DR): track 0.00 -> 118.5 mm, vias 0 -> 2
- net Net-(Q1-C): track 0.00 -> 109.5 mm, vias 0 -> 2
- net Net-(U1-THRE): track 25.7 -> 128.0 mm, vias 0 -> 4
- net AD9_3: track 100.7 -> 5.08 mm, vias 4 -> 2
- net Net-(U5-Q): track 11.4 -> 100.5 mm, vias 2 -> 4
- net AD10_3: track 92.9 -> 5.08 mm, vias 4 -> 2
- net M0RERD: track 0.00 -> 82.8 mm, vias 0 -> 3
- net M0DATR: track 0.00 -> 79.1 mm, vias 0 -> 1
- net M0THRE: track 0.00 -> 74.0 mm, vias 0 -> 1
- net AD11_3: track 78.9 -> 5.08 mm, vias 4 -> 2
- net AD6_3: track 76.2 -> 5.08 mm, vias 4 -> 2
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Other:
- board size 320 x 332.7 mm -> 320 x 327.7 mm

Commit message: 2026/1/15
Parts:
- removed C18: C, Capacitor_THT:C_Disc_D3.0mm_W1.6mm_P2.50mm
- removed Q10, Q11, Q12, Q8, Q9: NPN, Package_TO_SOT_THT:TO-92_Inline_Wide
- removed R17, R18, R19, R20, R21: 10k, Resistor_THT:R_Axial_DIN0207_L6.3mm_D2.5mm_P10.16mm_Horizontal
- added C20: 1u, Capacitor_THT:C_Disc_D3.0mm_W1.6mm_P2.50mm, F.Cu at (307.3, 233.6)
- added C21: C, Capacitor_THT:C_Disc_D3.0mm_W1.6mm_P2.50mm, F.Cu at (325.1, 208.3)
- added D13: D_Schottky, Diode_THT:D_DO-34_SOD68_P7.62mm_Horizontal, F.Cu at (325.1, 276.9)
- added D14: D_Schottky, Diode_THT:D_DO-34_SOD68_P7.62mm_Horizontal, F.Cu at (325.1, 274.3)
- added D15: D_Schottky, Diode_THT:D_DO-34_SOD68_P7.62mm_Horizontal, F.Cu at (325.1, 271.8)
- added D16: D_Schottky, Diode_THT:D_DO-34_SOD68_P7.62mm_Horizontal, F.Cu at (325.1, 269.2)
- added D17: D_Schottky, Diode_THT:D_DO-34_SOD68_P7.62mm_Horizontal, F.Cu at (325.1, 279.4)
- added D18: D, Diode_THT:D_DO-34_SOD68_P7.62mm_Horizontal, F.Cu at (284.5, 213.4)
- added D19: D_Schottky, Diode_THT:D_DO-34_SOD68_P7.62mm_Horizontal, F.Cu at (302.3, 254.0)
- added D20: D_Schottky, Diode_THT:D_DO-34_SOD68_P7.62mm_Horizontal, F.Cu at (294.6, 254.0)
- added J33: Conn_01x02_Pin, Connector_PinHeader_2.54mm:PinHeader_1x02_P2.54mm_Vertical, F.Cu at (345.4, 279.4)
- added J34: Conn_01x02_Pin, Connector_PinHeader_2.54mm:PinHeader_1x02_P2.54mm_Vertical, F.Cu at (315.0, 200.7)
- added Q4: NPN, Package_TO_SOT_THT:TO-92_Inline_Wide, F.Cu at (304.8, 205.7)
- added R12: 10k, Resistor_THT:R_Axial_DIN0207_L6.3mm_D2.5mm_P10.16mm_Horizontal, F.Cu at (307.3, 223.5)
- added R13: 1k, Resistor_THT:R_Axial_DIN0207_L6.3mm_D2.5mm_P10.16mm_Horizontal, F.Cu at (294.6, 210.8)
- added R9: 4.7k, Resistor_THT:R_Axial_DIN0207_L6.3mm_D2.5mm_P10.16mm_Horizontal, F.Cu at (320.0, 205.7)
- J31: value Conn_01x04_Pin -> Conn_01x12_Pin; footprint Connector_PinHeader_2.54mm:PinHeader_1x04_P2.54mm_Vertical -> Connector_PinHeader_2.54mm:PinHeader_1x12_P2.54mm_Vertical
- moved C8 237.0 mm to (368.3, 228.6)
- moved C15 236.3 mm to (345.4, 213.4)
- moved U10 234.2 mm to (355.6, 205.7), turned to 0 degrees
- moved C7 225.9 mm to (365.8, 215.9)
- moved RV2 217.7 mm to (365.8, 223.5), turned to 180 degrees
- moved R26 211.8 mm to (360.7, 218.4), turned to 0 degrees
- moved C16 203.2 mm to (281.9, 200.7), turned to 0 degrees
- moved R23 189.6 mm to (271.8, 208.3), turned to 180 degrees
- moved C10 189.1 mm to (360.7, 203.2), turned to 180 degrees
- moved C9 183.2 mm to (193.0, 129.5), turned to -90 degrees
- moved Q13 181.1 mm to (266.7, 200.7), turned to -90 degrees
- moved R22 179.0 mm to (279.4, 200.7)
- moved D2 178.3 mm to (274.3, 203.2)
- moved J29 173.0 mm to (251.5, 218.4)
- moved Q14 173.0 mm to (259.1, 210.8), turned to 90 degrees
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Connections:
- D10 pad 2: IRQ_1 -> IRQ_0
- J10 pad 1: IC1_1 -> IC1_0
- J11 pad 1: IC0_1 -> IC0_0
- J12 pad 1: Net-(J12-Pin_1) -> IC0_1
- J13 pad 1: Net-(J13-Pin_1) -> IC1_1
- J14 pad 1: Net-(J14-Pin_1) -> IC2_1
- J17 pad 1: IRQ_2 -> IRQ_1
- J17 pad 2: IC0_2 -> IC0_1
- J17 pad 3: IC1_2 -> IC1_1
- J17 pad 4: IC2_2 -> IC2_1
- J17 pad 5: IC3_2 -> IC3_1
- J28 pad 1: M0DATR -> M0STAT
- J28 pad 3: M0THRE -> /M0THL
- J28 pad 4: /M0THL -> /M0IQR
- J28 pad 5: /M0IQR -> unconnected-(J28-Pin_5-Pad5)
- J29 pad 10: /M1IQR -> unconnected-(J29-Pin_10-Pad10)
- J29 pad 5: unconnected-(J29-Pin_5-Pad5) -> M1STAT
- J29 pad 6: M1DATR -> M1RERD
- J29 pad 7: M1RERD -> /M1THL
- J29 pad 8: M1THRE -> /M1IQR
- J29 pad 9: /M1THL -> unconnected-(J29-Pin_9-Pad9)
- J30 pad 1: IC3_1 -> IC3_0
- J31 pad 1: Net-(J31-Pin_1) -> unconnected-(J31-Pin_1-Pad1)
- J31 pad 2: Net-(J31-Pin_2) -> unconnected-(J31-Pin_2-Pad2)
- J31 pad 3: Net-(J31-Pin_3) -> unconnected-(J31-Pin_3-Pad3)
- J31 pad 4: Net-(J31-Pin_4) -> unconnected-(J31-Pin_4-Pad4)
- J4 pad 1: IRQ_1 -> IRQ_0
- J4 pad 2: IC0_1 -> IC0_0
- J4 pad 3: IC1_1 -> IC1_0
- J4 pad 4: IC2_1 -> IC2_0
- J4 pad 5: IC3_1 -> IC3_0
- J9 pad 1: IC2_1 -> IC2_0
- U11 pad 11: Net-(J27-Pin_5) -> Net-(U11-O4)
- U11 pad 13: Net-(U11-O2) -> Net-(J27-Pin_3)
- U11 pad 7: Net-(U11-O7) -> Net-(J27-Pin_8)
- U11 pad 9: Net-(U11-O6) -> Net-(J27-Pin_7)
- U13 pad 10: Net-(J31-Pin_2) -> unconnected-(U13-O5-Pad10)
- U13 pad 11: Net-(J31-Pin_1) -> unconnected-(U13-O4-Pad11)
- U13 pad 7: Net-(J31-Pin_4) -> unconnected-(U13-O7-Pad7)
- U13 pad 9: Net-(J31-Pin_3) -> unconnected-(U13-O6-Pad9)
- U2 pad 1: Net-(U11-O0) -> Net-(U11-O4)
- U2 pad 10: Net-(J27-Pin_7) -> Net-(J27-Pin_2)
- U2 pad 11: Net-(U11-O6) -> Net-(U11-O1)
- U2 pad 12: Net-(J27-Pin_8) -> unconnected-(U2-Pad12)
- U2 pad 13: Net-(U11-O7) -> GND
- U2 pad 2: Net-(J27-Pin_1) -> Net-(J27-Pin_5)
- U2 pad 3: Net-(U11-O1) -> Net-(U11-O5)
- U2 pad 4: Net-(J27-Pin_2) -> Net-(J27-Pin_6)
- U2 pad 5: Net-(U11-O2) -> GND
- U2 pad 6: Net-(J27-Pin_3) -> unconnected-(U2-Pad6)
- U2 pad 8: Net-(J27-Pin_6) -> Net-(J27-Pin_1)
- U2 pad 9: Net-(U11-O5) -> Net-(U11-O0)
- U6 pad 10: M0DATR -> M0STAT
- U6 pad 2: M0THRE -> M0STAT
- U7 pad 18: /DRR2 -> /M1IQR
- U7 pad 2: -12V -> Net-(J34-Pin_1)
- U7 pad 23: /THRL2 -> /M1THL
- U7 pad 4: RRD2 -> M1RERD
- U8 pad 10: GND -> M1STAT
- U8 pad 11: unconnected-(U8-Pad11) -> Net-(D13-K)
- U8 pad 12: GND -> Net-(U8-Pad12)
- U8 pad 13: GND -> /M1IQR
- U8 pad 2: THRE2 -> M1STAT
- U8 pad 3: Net-(U8-Pad3) -> Net-(D19-K)
- U8 pad 4: Net-(U8-Pad3) -> Net-(Q4-C)
- U8 pad 5: Net-(U8-Pad3) -> Net-(D13-K)
- U8 pad 6: Net-(R21-Pad1) -> Net-(U8-Pad12)
- U8 pad 8: unconnected-(U8-Pad8) -> Net-(D20-K)
- U8 pad 9: GND -> Net-(U7-DR)
- U9 pad 11: unconnected-(U9-Pad11) -> Net-(R12-Pad1)
- U9 pad 12: GND -> Net-(U7-DR)
- U9 pad 13: GND -> Net-(D18-K)
Routing:
- net +5V: track 825.1 -> 1300.4 mm, vias 26 -> 33
- net GND: track 882.6 -> 1255.0 mm, vias 26 -> 41
- net /THRL2: track 211.3 -> 0.00 mm, vias 6 -> 0
- net /M1THL: track 0.00 -> 164.4 mm, vias 0 -> 4
- net AD4_3: track 5.08 -> 158.3 mm, vias 2 -> 5
- net AD3_3: track 5.08 -> 130.6 mm, vias 2 -> 5
- net AD2_3: track 5.08 -> 129.3 mm, vias 2 -> 5
- net AD1_3: track 5.08 -> 127.9 mm, vias 2 -> 5
- net Net-(D11-K): track 0.00 -> 119.7 mm, vias 0 -> 8
- net M0STAT: track 0.00 -> 114.8 mm, vias 0 -> 3
- net /M1IQR: track 0.00 -> 112.2 mm, vias 0 -> 2
- net Net-(Q4-C): track 0.00 -> 109.5 mm, vias 0 -> 2
- net Net-(J27-Pin_4): track 0.00 -> 108.3 mm, vias 0 -> 3
- net Net-(J27-Pin_7): track 0.00 -> 107.1 mm, vias 0 -> 3
- net M1STAT: track 0.00 -> 102.1 mm, vias 0 -> 2
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Other:
- board size 320 x 327.7 mm -> 309.9 x 203.2 mm
