File: KiCad FIles/TMSHB_UART_ALL_V2/TMSHB_UART_ALL_V2.kicad_sch (KiCad schematic)
At the start: 99 parts, among them J1 Conn_01x08_Pin, J10 Conn_01x02_Pin, J11 Conn_01x02_Pin, J12 Conn_01x02_Pin, J13 Conn_01x02_Pin, J14 Conn_01x02_Pin, J15 Conn_01x16_Pin, J16 Conn_01x08_Pin, J17 Conn_01x05_Pin, J18 Conn_01x05_Pin, J19 Conn_01x05_Pin, J2 Conn_01x15_Pin, J20 Conn_01x15_Pin, J21 Conn_01x15_Pin, J22 Conn_01x16_Pin, J23 Conn_01x08_Pin, J24 Conn_01x05_Pin, J25 Conn_01x05_Pin, J26 Conn_01x05_Pin, J27 Conn_01x12_Pin, J28 Conn_01x12_Pin, J29 Conn_01x12_Pin, J3 Conn_01x16_Pin, J4 Conn_01x05_Pin, J5 Conn_01x05_Pin, J6 Conn_01x03_Pin, J7 Conn_01x05_Pin, J8 Conn_01x03_Pin, J9 Conn_01x02_Pin, Q1 NPN, Q10 NPN, Q11 NPN, Q12 NPN, Q13 NPN, Q14 PNP, Q2 PNP, Q3 NPN, Q4 NPN, Q5 NPN, Q6 NPN, Q7 NPN, Q8 NPN, Q9 NPN, U1 TR1602, U10 NE555P, U11 74LS138, U12 74LS32, U2 27C16, U3 74LS00, U4 74LS32, U5 NE555P, U6 74LS00, U7 TR1602, U8 74LS00, U9 74LS32

Commit message: 2026/1/13
Parts:
- removed Q4, Q5, Q6, Q7: NPN, Package_TO_SOT_THT:TO-92_Inline_Wide, symbol Simulation_SPICE:NPN
- removed R12, R13, R14, R15: 10k, Resistor_THT:R_Axial_DIN0207_L6.3mm_D2.5mm_P10.16mm_Horizontal, symbol Device:R
- added C19: 1u, Capacitor_THT:C_Disc_D3.0mm_W1.6mm_P2.50mm, symbol Device:C
- added D10, D4, D5, D6, D7, D8, D9: D_Schottky, Diode_THT:D_DO-34_SOD68_P7.62mm_Horizontal, symbol Device:D_Schottky
- added D3: D, Diode_THT:D_DO-34_SOD68_P7.62mm_Horizontal, symbol Device:D
- added J30: Conn_01x02_Pin, Connector_PinHeader_2.54mm:PinHeader_1x02_P2.54mm_Vertical, symbol Connector:Conn_01x02_Pin
- added J31, J32: Conn_01x08_Pin, symbol Connector:Conn_01x08_Pin
- added R1: 4.7k, Resistor_THT:R_Axial_DIN0207_L6.3mm_D2.5mm_P10.16mm_Horizontal, symbol Device:R
- added R2: 1k, Resistor_THT:R_Axial_DIN0207_L6.3mm_D2.5mm_P10.16mm_Horizontal, symbol Device:R
- added U13: 74LS138, Package_DIP:DIP-16_W7.62mm, symbol 74xx:74LS138
Connections:
- net +5V: now also R1.1, U13.16 (VCC), U13.6 (E3)
- net DA0_1: now also D4.2 (A); no longer Q1.1 (C)
- net DA1_1: now also D5.2 (A)
- net GND: now also D3.2 (A), R2.1, U13.8 (GND); no longer U4.12, U4.13, U6.10, U6.12, U6.13, U6.9
- net IC0_1: now also J11.1 (Pin_1)
- net IC1_1: now also J10.1 (Pin_1)
- net IC2_1: now also J9.1 (Pin_1)
- net IC3_1: now also J30.1 (Pin_1)
- net IRQ_1: now also D10.2 (A)
- net RRD1: no longer J27.3 (Pin_3)
- net RRD2: no longer J28.7 (Pin_7)
- net THRE1: no longer J27.1 (Pin_1)
- net THRE2: no longer J28.5 (Pin_5)
- net /DRR1: no longer J27.4 (Pin_4)
- net /DRR2: no longer J28.8 (Pin_8)
- net /THRL1: no longer J27.2 (Pin_2)
- net /THRL2: no longer J28.6 (Pin_6)
- net at U3.8: no longer J29.1 (Pin_1)
- net at R5.1: now also U4.11; no longer U6.6
- net at U1.19 (DR): now also U4.12, U6.9
- net at U1.22 (THRE), U6.1: now also C19.1
- net at J11.2 (Pin_2): now also D6.2 (A)
- net at U3.11: no longer J29.5 (Pin_5)
- net at J10.2 (Pin_2): now also D7.2 (A)
- net at J29.2 (Pin_2): no longer U11.14 (O1)
- net at J29.3 (Pin_3): no longer U11.13 (O2)
- net at J29.4 (Pin_4): no longer U11.12 (O3)
- net at J29.6 (Pin_6): no longer U11.10 (O5)
- net at J29.7 (Pin_7): no longer U11.9 (O6)
- net at J29.8 (Pin_8): no longer U11.7 (O7)
- net at J9.2 (Pin_2): now also D8.2 (A)
- net at U2.9 (D0): now also J31.1 (Pin_1); no longer U11.1 (A0)
- net at U2.10 (D1): now also J31.2 (Pin_2); no longer U11.2 (A1)
- net at U2.11 (D2): now also J31.3 (Pin_3); no longer U11.3 (A2)
- net at U11.4 (E1), U11.5 (E2): now also J32.8 (Pin_8), U13.4 (E1), U13.5 (E2); no longer U12.11, U2.20 (~{OE})
- net at U6.8: now also D5.1 (K)
- net at U2.13 (D3): now also J31.4 (Pin_4)
- net at U2.14 (D4): now also J31.5 (Pin_5)
- net at U2.15 (D5): now also J31.6 (Pin_6)
- net at U6.11: now also U6.5, D10.1 (K), D6.1 (K), D7.1 (K), D8.1 (K), D9.1 (K)
- new net: D4.1 (K), U6.3
- new net: J32.4 (Pin_4), U13.1 (A0)
- new net: J32.5 (Pin_5), U13.2 (A1)
- new net: J32.6 (Pin_6), U13.3 (A2)
- new net: J31.8 (Pin_8), U12.11, U2.20 (~{OE})
- new net: D9.2 (A), J30.2 (Pin_2)
- new net: C19.2, D3.1 (K), R2.2, U4.13
- new net: J32.1 (Pin_1), U11.1 (A0)
- new net: J32.2 (Pin_2), U11.2 (A1)
- new net: J32.3 (Pin_3), U11.3 (A2)
- new net: Q1.1 (C), R1.2, U6.4
- new net: U6.12, U6.6
- new net DR1: U6.10
- new net /IRQRST1: U6.13
- now unconnected: U11.11 (O4), U11.15 (O0), U3.10, U3.12, U3.13, U3.9
Other:
- moved on the sheet: J27, J28, J29, U10, U11, U12A, U12B, U12C, U12D, U12E, U2, U3A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

Commit message: 2026/1/13
Parts:
- removed J31, J32: Conn_01x08_Pin, symbol Connector:Conn_01x08_Pin
- removed U12: 74LS32, Package_DIP:DIP-14_W7.62mm, symbol 74xx:74LS32
- removed U2: 27C16, Package_DIP:DIP-24_W15.24mm, symbol User:27C16
- added D11, D12: D_Schottky, Diode_THT:D_DO-34_SOD68_P7.62mm_Horizontal, symbol Device:D_Schottky
- added J31: Conn_01x04_Pin, Connector_PinHeader_2.54mm:PinHeader_1x04_P2.54mm_Vertical, symbol Connector:Conn_01x04_Pin
- added J32: Conn_01x02_Pin, Connector_PinHeader_2.54mm:PinHeader_1x02_P2.54mm_Vertical, symbol Connector:Conn_01x02_Pin
- added R8: 1k, Resistor_THT:R_Axial_DIN0207_L6.3mm_D2.5mm_P10.16mm_Horizontal, symbol Device:R
- added U2: 74LS04, Package_DIP:DIP-14_W7.62mm, symbol 74xx:74LS04
- J27, J28, J29: footprint Connector_PinSocket_2.54mm:PinSocket_1x12_P2.54mm_Vertical -> Connector_PinHeader_2.54mm:PinHeader_1x12_P2.54mm_Vertical
Connections:
- net DR1 is gone; now on net M0DATR: U6.10
- net RRD1 is gone; now on net M0RERD: U1.4 (RRD)
- net THRE1 is gone; now on net M0THRE: U6.2
- net /DRR1 is gone; now on net /M0IQR: U1.18 (DRR)
- net /IRQRST1 is gone; now on net /M0IQR: U6.13
- net /THRL1 is gone; now on net /M0THL: U1.23 (THRL)
- net +5V: now also U2.14 (VCC)
- net -12V: now also J32.2 (Pin_2); no longer C17.1, U1.2 (-12V)
- net AD1_3: now also U11.1 (A0), U13.1 (A0)
- net AD2_3: now also U11.2 (A1), U13.2 (A1)
- net AD3_3: now also U11.3 (A2), U13.3 (A2)
- net AD4_3: now also U11.5 (E2), U3.10, U3.9
- net GND: now also U3.12, U3.13, R8.1, U2.7 (GND)
- net M0DATR: now reaches J28.1 (Pin_1)
- net M0RERD: now reaches J28.2 (Pin_2)
- net M0THRE: now reaches J28.3 (Pin_3)
- net /M0THL: now reaches J28.4 (Pin_4)
- net /M0IQR: now reaches J28.5 (Pin_5)
- net at U3.8: now also U13.5 (E2)
- net at U13.10 (O5): now also J31.2 (Pin_2)
- net at U13.11 (O4): now also J31.1 (Pin_1)
- net at U13.12 (O3): now also J27.12 (Pin_12)
- net at U13.13 (O2): now also J27.11 (Pin_11)
- net at U13.14 (O1): now also J27.10 (Pin_10)
- net at U13.15 (O0): now also J27.9 (Pin_9)
- net at U11.4 (E1), U13.4 (E1): now also D11.1 (K), D12.1 (K), R8.2; no longer U11.5 (E2), U13.5 (E2)
- net at U13.7 (O7): now also J31.4 (Pin_4)
- net at U13.9 (O6): now also J31.3 (Pin_3)
- net /M1IQR: now reaches J29.10 (Pin_10)
- net M1DATR: now reaches J29.6 (Pin_6)
- net M1RERD: now reaches J29.7 (Pin_7)
- net M1THRE: now reaches J29.8 (Pin_8)
- net /M1THL: now reaches J29.9 (Pin_9)
- net at U11.10 (O5): now also U2.9
- net at U11.11 (O4): now also J27.5 (Pin_5)
- net at U11.12 (O3): now also J27.4 (Pin_4)
- net at U11.13 (O2): now also U2.5
- net at U11.14 (O1): now also U2.3
- net at U11.15 (O0): now also U2.1
- net at U11.7 (O7): now also U2.13
- net at U11.9 (O6): now also U2.11
- net at U3.3: now also D11.2 (A)
- net at U3.6: now also D12.2 (A)
- net at J27.1 (Pin_1): now also U2.2
- net at J27.2 (Pin_2): now also U2.4
- net at J27.3 (Pin_3): now also U2.6
- net at J27.6 (Pin_6): now also U2.8
- net at J27.7 (Pin_7): now also U2.10
- net at J27.8 (Pin_8): now also U2.12
- new net: C17.1, J32.1 (Pin_1), U1.2 (-12V)
Other:
- moved on the sheet: U11, U13, U3C, U3D

Commit message: 2026/1/15
Parts:
- removed C18: C, Capacitor_THT:C_Disc_D3.0mm_W1.6mm_P2.50mm, symbol Device:C
- removed J31: Conn_01x04_Pin, Connector_PinHeader_2.54mm:PinHeader_1x04_P2.54mm_Vertical, symbol Connector:Conn_01x04_Pin
- removed Q10, Q11, Q12, Q8, Q9: NPN, Package_TO_SOT_THT:TO-92_Inline_Wide, symbol Simulation_SPICE:NPN
- removed R17, R18, R19, R20, R21: 10k, Resistor_THT:R_Axial_DIN0207_L6.3mm_D2.5mm_P10.16mm_Horizontal, symbol Device:R
- added C20: 1u, Capacitor_THT:C_Disc_D3.0mm_W1.6mm_P2.50mm, symbol Device:C
- added C21: C, Capacitor_THT:C_Disc_D3.0mm_W1.6mm_P2.50mm, symbol Device:C
- added D13, D14, D15, D16, D17, D19, D20: D_Schottky, Diode_THT:D_DO-34_SOD68_P7.62mm_Horizontal, symbol Device:D_Schottky
- added D18: D, Diode_THT:D_DO-34_SOD68_P7.62mm_Horizontal, symbol Device:D
- added J31: Conn_01x12_Pin, Connector_PinHeader_2.54mm:PinHeader_1x12_P2.54mm_Vertical, symbol Connector:Conn_01x12_Pin
- added J33, J34: Conn_01x02_Pin, Connector_PinHeader_2.54mm:PinHeader_1x02_P2.54mm_Vertical, symbol Connector:Conn_01x02_Pin
- added J35: Conn_01x14_Pin, symbol Connector:Conn_01x14_Pin
- added Q4: NPN, Package_TO_SOT_THT:TO-92_Inline_Wide, symbol Simulation_SPICE:NPN
- added R12: 10k, Resistor_THT:R_Axial_DIN0207_L6.3mm_D2.5mm_P10.16mm_Horizontal, symbol Device:R
- added R13: 1k, Resistor_THT:R_Axial_DIN0207_L6.3mm_D2.5mm_P10.16mm_Horizontal, symbol Device:R
- added R9: 4.7k, Resistor_THT:R_Axial_DIN0207_L6.3mm_D2.5mm_P10.16mm_Horizontal, symbol Device:R
Connections:
- net IC0_2 is gone; now on net IC0_1: J17.2 (Pin_2)
- net IC1_2 is gone; now on net IC1_1: J17.3 (Pin_3)
- net IC2_2 is gone; now on net IC2_1: J17.4 (Pin_4)
- net IC3_2 is gone; now on net IC3_1: J17.5 (Pin_5)
- net IRQ_2 is gone; now on net IRQ_1: J17.1 (Pin_1)
- net M1DATR is gone; now on net M1RERD: J29.6 (Pin_6)
- net M1THRE is gone; now on net /M1IQR: J29.8 (Pin_8)
- net RRD2 is gone; now on net M1RERD: U7.4 (RRD)
- net THRE2 is gone; now on net M1STAT: U8.2
- net /DRR2 is gone; now on net /M1IQR: U7.18 (DRR)
- net /THRL2 is gone; now on net /M1THL: U7.23 (THRL)
- net +5V: now also R9.1
- net -12V: now also J34.2 (Pin_2); no longer U7.2 (-12V)
- net DA0_1: now also D19.2 (A)
- net DA1_1: now also D20.2 (A)
- net GND: now also U2.13, U2.5, C21.2, D18.2 (A), J35.1 (Pin_1), Q4.3 (E), R13.1; no longer U8.10, U8.12, U8.13, U8.9, U9.12, U9.13
- net IC0_1: now also J12.1 (Pin_1); no longer J11.1 (Pin_1), J4.2 (Pin_2)
- net IC1_1: now also J13.1 (Pin_1); no longer J10.1 (Pin_1), J4.3 (Pin_3)
- net IC2_1: now also J14.1 (Pin_1); no longer J4.4 (Pin_4), J9.1 (Pin_1)
- net IC3_1: now also J33.1 (Pin_1); no longer J30.1 (Pin_1), J4.5 (Pin_5)
- net IRQ_1: now also D17.2 (A); no longer D10.2 (A), J4.1 (Pin_1)
- net M1RERD: no longer J29.7 (Pin_7)
- net PBUSY: now also J31.10 (Pin_10)
- net PSTRB: now also J31.12 (Pin_12)
- net /M0IQR: now also J28.4 (Pin_4); no longer J28.5 (Pin_5)
- net /M0THL: now also J28.3 (Pin_3); no longer J28.4 (Pin_4)
- net /M1IQR: now also U8.13; no longer J29.10 (Pin_10)
- net /M1THL: now also J29.7 (Pin_7); no longer J29.9 (Pin_9)
- net /PACK: now also J31.9 (Pin_9)
- net /PPRF: now also J31.11 (Pin_11)
- net at U2.10: now also J27.2 (Pin_2); no longer J27.7 (Pin_7)
- net at U2.11: now also U11.14 (O1); no longer U11.9 (O6)
- net at U7.19 (DR): now also U8.9, U9.12
- net at J14.2 (Pin_2): now also D15.2 (A)
- net at J13.2 (Pin_2): now also D14.2 (A)
- net M1STAT: now reaches J29.5 (Pin_5)
- net M1STAT: now also U8.10
- net at U8.8: now also D20.1 (K)
- net at U11.13 (O2): now also J27.3 (Pin_3); no longer U2.5
- net at U2.6: no longer J27.3 (Pin_3)
- net at U9.11: now also R12.1
- net at U7.22 (THRE), U8.1: now also C20.1
- net at U8.11: now also U8.5, D13.1 (K), D14.1 (K), D15.1 (K), D16.1 (K), D17.1 (K)
- net at J27.1 (Pin_1): now also U2.8; no longer U2.2
- net at U2.4: now also J27.6 (Pin_6); no longer J27.2 (Pin_2)
- net at J27.5 (Pin_5): now also U2.2; no longer U11.11 (O4)
- net at J27.8 (Pin_8): now also U11.7 (O7); no longer U2.12
- net at J12.2 (Pin_2): now also D13.2 (A)
- net at U2.1: now also U11.11 (O4); no longer U11.15 (O0)
- net at U11.10 (O5): now also U2.3; no longer U2.9
- net at U8.6: now also U8.12
- net M0DATR renamed M0STAT
- net M0STAT: now also U6.2
- removed net M0THRE: J28.3 (Pin_3), U6.2
- new net: Q4.1 (C), R9.2, U8.4
- new net: Q4.2 (B), R12.2
- new net: C20.2, D18.1 (K), R13.2, U9.13
- new net: C21.1, J34.1 (Pin_1), U7.2 (-12V)
- new net: D16.2 (A), J33.2 (Pin_2)
- new net: J27.7 (Pin_7), U11.9 (O6)
- new net: U11.15 (O0), U2.9
- new net: D19.1 (K), U8.3
- new net DA0_3: J35.3 (Pin_3)
- new net DA1_3: J35.4 (Pin_4)
- new net DA2_3: J35.5 (Pin_5)
- new net DA3_3: J35.6 (Pin_6)
- new net DA4_3: J35.7 (Pin_7)
- new net DA5_3: J35.8 (Pin_8)
- new net DA6_3: J35.9 (Pin_9)
- new net DA7_3: J35.10 (Pin_10)
- new net IC0_0: J11.1 (Pin_1), J4.2 (Pin_2)
- new net IC1_0: J10.1 (Pin_1), J4.3 (Pin_3)
- new net IC2_0: J4.4 (Pin_4), J9.1 (Pin_1)
- new net IC3_0: J30.1 (Pin_1), J4.5 (Pin_5)
- new net IRQ_0: D10.2 (A), J4.1 (Pin_1)
Other:
- moved on the sheet: U10, U2A, U2B, U2C, U2D, U2E, U2F, U7, U8A, U8B, U8C, U8D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
