File: KiCad FIles/TMSHB_BUFF/TMSHB_BUFF.kicad_sch (KiCad schematic)
At the start: 16 parts, among them J1 Conn_01x08_Pin, J10 Conn_01x05_Pin, J11 Conn_01x05_Pin, J12 Conn_01x05_Pin, J2 Conn_01x15_Pin, J3 Conn_01x16_Pin, J4 Conn_01x05_Pin, J5 Conn_01x16_Pin, J6 Conn_01x15_Pin, J7 Conn_01x08_Pin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

Commit message: 2026/4/9
Other:
- moved on the sheet: J1, J7
Changed lines of the file:
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@@
 	)
 	(junction
-		(at 99.06 170.18)
+		(at 99.06 149.86)
 		(diameter 0)
 		(color 0 0 0 0)
@@
 	(wire
 		(pts
-			(xy 74.93 180.34) (xy 123.19 180.34)
+			(xy 74.93 160.02) (xy 123.19 160.02)
 		)
 		(stroke
@@
 	(wire
 		(pts
-			(xy 99.06 170.18) (xy 123.19 170.18)
+			(xy 99.06 149.86) (xy 123.19 149.86)
 		)
 		(stroke
@@
 	(wire
 		(pts
-			(xy 99.06 118.11) (xy 99.06 170.18)
+			(xy 99.06 118.11) (xy 99.06 149.86)
 		)
 		(stroke
@@
 	(wire
 		(pts
-			(xy 74.93 177.8) (xy 123.19 177.8)
+			(xy 74.93 157.48) (xy 123.19 157.48)
 		)
 		(stroke
@@
 	(wire
 		(pts
-			(xy 74.93 187.96) (xy 123.19 187.96)
+			(xy 74.93 167.64) (xy 123.19 167.64)
 		)
 		(stroke
@@
 	(wire
 		(pts
-			(xy 74.93 182.88) (xy 123.19 182.88)
+			(xy 74.93 162.56) (xy 123.19 162.56)
 		)
 		(stroke
@@
 	(wire
 		(pts
-			(xy 74.93 172.72) (xy 123.19 172.72)
+			(xy 74.93 152.4) (xy 123.19 152.4)
 		)
 		(stroke
@@
 	(wire
 		(pts
-			(xy 99.06 170.18) (xy 74.93 170.18)
+			(xy 99.06 149.86) (xy 74.93 149.86)
 		)
 		(stroke
@@
 	(wire
 		(pts
-			(xy 74.93 185.42) (xy 123.19 185.42)
+			(xy 74.93 165.1) (xy 123.19 165.1)
 		)
 		(stroke
@@
 	(wire
 		(pts
-			(xy 74.93 175.26) (xy 123.19 175.26)
+			(xy 74.93 154.94) (xy 123.19 154.94)
 		)
 		(stroke
@@
 	)
 	(label "{slash}HOLD"
-		(at 115.57 180.34 0)
+		(at 115.57 160.02 0)
 		(effects
 			(font
@@
 	)
 	(label "READY"
-		(at 115.57 175.26 0)
+		(at 115.57 154.94 0)
 		(effects
 			(font
@@
 	)
 	(label "{slash}MEMIN"
-		(at 115.57 172.72 0)
+		(at 115.57 152.4 0)
 		(effects
 			(font
@@
 	)
 	(label "DBIN"
-		(at 115.57 170.18 0)
+		(at 115.57 149.86 0)
 		(effects
 			(font
@@
 	)
 	(label "{slash}WE"
-		(at 82.55 177.8 180)
+		(at 82.55 157.48 180)
 		(effects
 			(font
@@
 	)
 	(label "DBIN"
-		(at 82.55 170.18 180)
+		(at 82.55 149.86 180)
 		(effects
 			(font
@@
 	)
 	(label "{slash}WE"
-		(at 115.57 177.8 0)
+		(at 115.57 157.48 0)
 		(effects
 			(font
@@
 	)
 	(label "HOLDA"
-		(at 82.55 185.42 180)
+		(at 82.55 165.1 180)
 		(effects
 			(font
@@
 	)
 	(label "HOLDA"
-		(at 115.57 185.42 0)
+		(at 115.57 165.1 0)
 		(effects
 			(font
@@
 	)
 	(label "WAIT"
-		(at 115.57 182.88 0)
+		(at 115.57 162.56 0)
 		(effects
 			(font
@@
 	)
 	(label "{slash}HOLD"
-		(at 82.55 180.34 180)
+		(at 82.55 160.02 180)
 		(effects
 			(font
@@
 	)
 	(label "READY"
-		(at 82.55 175.26 180)
+		(at 82.55 154.94 180)
 		(effects
 			(font
@@
 	)
 	(label "WAIT"
-		(at 82.55 182.88 180)
+		(at 82.55 162.56 180)
 		(effects
 			(font
@@
 	)
 	(label "{slash}MEMIN"
-		(at 82.55 172.72 180)
+		(at 82.55 152.4 180)
 		(effects
 			(font
@@
 	)
 	(label "{slash}RESET"
-		(at 115.57 187.96 0)
+		(at 115.57 167.64 0)
 		(effects
 			(font
@@
 	)
 	(label "{slash}RESET"
-		(at 82.55 187.96 180)
+		(at 82.55 167.64 180)
 		(effects
 			(font
@@
 		)
 		(instances
-			(project ""
+			(project "TMSHB_BUFF"
 				(path "/0f639dad-2718-4cff-a122-33c660513b27"
 					(reference "U1")
@@
 	(symbol
 		(lib_id "Connector:Conn_01x08_Pin")
-		(at 128.27 177.8 0)
+		(at 128.27 157.48 0)
 		(mirror y)
 		(unit 1)
@@
 		(dnp no)
 		(property "Reference" "J1"
-			(at 128.27 168.148 0)
+			(at 128.27 147.828 0)
 			(effects
 				(font
@@
 		)
 		(property "Value" "Conn_01x08_Pin"
-			(at 127.635 167.64 0)
+			(at 127.635 147.32 0)
 			(effects
 				(font
@@
 		)
 		(property "Footprint" "Connector_PinHeader_2.54mm:PinHeader_1x08_P2.54mm_Vertical"
-			(at 128.27 177.8 0)
+			(at 128.27 157.48 0)
 			(effects
 				(font
@@
 		)
 		(property "Datasheet" "~"
-			(at 128.27 177.8 0)
+			(at 128.27 157.48 0)
 			(effects
 				(font
@@
 		)
 		(property "Description" "Generic connector, single row, 01x08, script generated"
-			(at 128.27 177.8 0)
+			(at 128.27 157.48 0)
 			(effects
 				(font
@@
 	(symbol
 		(lib_id "Connector:Conn_01x08_Pin")
-		(at 69.85 177.8 0)
+		(at 69.85 157.48 0)
 		(unit 1)
 		(exclude_from_sim no)
@@
 		(dnp no)
 		(property "Reference" "J7"
-			(at 69.85 168.148 0)
+			(at 69.85 147.828 0)
 			(effects
 				(font
@@
 		)
 		(property "Value" "Conn_01x08_Pin"
-			(at 70.485 167.64 0)
+			(at 70.485 147.32 0)
 			(effects
 				(font
@@
 		)
 		(property "Footprint" "Connector_PinHeader_2.54mm:PinHeader_1x08_P2.54mm_Vertical"
-			(at 69.85 177.8 0)
+			(at 69.85 157.48 0)
 			(effects
 				(font
@@
 		)
 		(property "Datasheet" "~"
-			(at 69.85 177.8 0)
+			(at 69.85 157.48 0)
 			(effects
 				(font
@@
 		)
 		(property "Description" "Generic connector, single row, 01x08, script generated"
-			(at 69.85 177.8 0)
+			(at 69.85 157.48 0)
 			(effects
 				(font
