File: KiCad FIles/!Old/TMSHB_BUFF/TMSHB_BUFF.kicad_pcb (KiCad board)
At the start: 2 copper layers, 149.9 x 73.7 mm, 28 parts, among them J1 Conn_01x08_Pin, J10 Conn_01x05_Pin, J11 Conn_01x05_Pin, J12 Conn_01x05_Pin, J2 Conn_01x15_Pin, J3 Conn_01x16_Pin, J4 Conn_01x05_Pin, J5 Conn_01x16_Pin, J6 Conn_01x15_Pin, J7 Conn_01x08_Pin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

Commit message: 2026/6/10
Parts:
- removed the J1 at (114.3, 94.0)
- removed the J10 at (63.5, 55.9)
- removed the J10 at (63.5, 94.0)
- removed the J11 at (50.8, 73.7)
- removed the J11 at (50.8, 35.6)
- removed the J12 at (63.5, 73.7)
- removed the J12 at (63.5, 35.6)
- removed the J2 at (76.2, 94.0)
- removed the J7 at (114.3, 73.7)
- removed the J9 at (50.8, 55.9)
- removed the J9 at (50.8, 94.0)
- added J10: Conn_01x05_Pin, Connector_PinHeader_2.54mm:PinHeader_1x05_P2.54mm_Vertical, F.Cu at (63.5, 73.7)
- added J10: Conn_01x05_Pin, Connector_PinHeader_2.54mm:PinHeader_1x05_P2.54mm_Vertical, F.Cu at (63.5, 35.6)
- added J11: Conn_01x05_Pin, Connector_PinHeader_2.54mm:PinHeader_1x05_P2.54mm_Vertical, F.Cu at (50.8, 94.0)
- added J12: Conn_01x05_Pin, Connector_PinHeader_2.54mm:PinHeader_1x05_P2.54mm_Vertical, F.Cu at (63.5, 55.9)
- added J12: Conn_01x05_Pin, Connector_PinHeader_2.54mm:PinHeader_1x05_P2.54mm_Vertical, F.Cu at (63.5, 94.0)
- added J13: Conn_01x05_Pin, Connector_PinHeader_2.54mm:PinHeader_1x05_P2.54mm_Vertical, F.Cu at (50.8, 55.9)
- added J14: Conn_01x05_Pin, Connector_PinHeader_2.54mm:PinHeader_1x05_P2.54mm_Vertical, F.Cu at (50.8, 35.6)
- added J15: Conn_01x08_Pin, Connector_PinHeader_2.54mm:PinHeader_1x08_P2.54mm_Vertical, F.Cu at (114.3, 94.0)
- added J16: Conn_01x08_Pin, Connector_PinHeader_2.54mm:PinHeader_1x08_P2.54mm_Vertical, F.Cu at (114.3, 73.7)
- added J6: Conn_01x15_Pin, Connector_PinHeader_2.54mm:PinHeader_1x15_P2.54mm_Vertical, F.Cu at (76.2, 94.0)
- added J9: Conn_01x05_Pin, Connector_PinHeader_2.54mm:PinHeader_1x05_P2.54mm_Vertical, F.Cu at (50.8, 73.7)
Connections:
- J6 pad 1: /BAD1 -> (no net)
- J6 pad 10: /BAD10 -> (no net)
- J6 pad 11: /BAD11 -> (no net)
- J6 pad 12: /BAD12 -> (no net)
- J6 pad 13: /BAD13 -> (no net)
- J6 pad 14: /BAD14 -> (no net)
- J6 pad 15: /BAD15 -> (no net)
- J6 pad 2: /BAD2 -> (no net)
- J6 pad 3: /BAD3 -> (no net)
- J6 pad 4: /BAD4 -> (no net)
- J6 pad 5: /BAD5 -> (no net)
- J6 pad 6: /BAD6 -> (no net)
- J6 pad 7: /BAD7 -> (no net)
- J6 pad 8: /BAD8 -> (no net)
- J6 pad 9: /BAD9 -> (no net)
- U3 pad 1: +5V -> GND
- U4 pad 1: +5V -> GND
Routing:
- net GND: track 327.7 -> 361.2 mm, vias 5 -> 8
- net +5V: track 290.0 -> 262.1 mm, vias 14 -> 10
- net (no net): vias 1 -> 0
