File: KiCad FIles/TMSHB_ADDR_BUFF/TMSHB_ADDR_BUFF.kicad_sch (KiCad schematic)
At the start: 16 parts, among them J1 Conn_01x08_Pin, J10 Conn_01x05_Pin, J11 Conn_01x05_Pin, J12 Conn_01x05_Pin, J2 Conn_01x15_Pin, J3 Conn_01x16_Pin, J4 Conn_01x05_Pin, J5 Conn_01x16_Pin, J6 Conn_01x15_Pin, J7 Conn_01x08_Pin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

Commit message: 2026/6/10
Parts:
- removed J10, J12: Conn_01x05_Pin, Connector_PinHeader_2.54mm:PinHeader_1x05_P2.54mm_Vertical, symbol Connector:Conn_01x05_Pin
- removed J2, J6: Conn_01x15_Pin, Connector_PinHeader_2.54mm:PinHeader_1x15_P2.54mm_Vertical, symbol Connector:Conn_01x15_Pin
- removed U1, U2: 74LS245, Package_DIP:DIP-20_W7.62mm, symbol 74xx:74LS245
- added C1, C2: C, Capacitor_THT:C_Disc_D3.0mm_W1.6mm_P2.50mm, symbol Device:C
- added J13, J14: Conn_01x08_Pin, Connector_PinHeader_2.54mm:PinHeader_1x08_P2.54mm_Vertical, symbol Connector:Conn_01x08_Pin
- added J15, J16: Conn_01x05_Pin, Connector_PinHeader_2.54mm:PinHeader_1x05_P2.54mm_Vertical, symbol Connector:Conn_01x05_Pin
- added J2, J6: Conn_01x07_Pin, Connector_PinHeader_2.54mm:PinHeader_1x07_P2.54mm_Vertical, symbol Connector:Conn_01x07_Pin
Connections:
- net DA0 is gone; now on net BDA0: J3.1 (Pin_1)
- net DA1 is gone; now on net BDA1: J3.2 (Pin_2)
- net DA10 is gone; now on net BDA10: J3.11 (Pin_11)
- net DA11 is gone; now on net BDA11: J3.12 (Pin_12)
- net DA12 is gone; now on net BDA12: J3.13 (Pin_13)
- net DA13 is gone; now on net BDA13: J3.14 (Pin_14)
- net DA14 is gone; now on net BDA14: J3.15 (Pin_15)
- net DA15 is gone; now on net BDA15: J3.16 (Pin_16)
- net DA2 is gone; now on net BDA2: J3.3 (Pin_3)
- net DA3 is gone; now on net BDA3: J3.4 (Pin_4)
- net DA4 is gone; now on net BDA4: J3.5 (Pin_5)
- net DA5 is gone; now on net BDA5: J3.6 (Pin_6)
- net DA6 is gone; now on net BDA6: J3.7 (Pin_7)
- net DA7 is gone; now on net BDA7: J3.8 (Pin_8)
- net DA8 is gone; now on net BDA8: J3.9 (Pin_9)
- net DA9 is gone; now on net BDA9: J3.10 (Pin_10)
- net +12V: now also J15.1 (Pin_1), J16.1 (Pin_1)
- net +5V: now also C1.1, C2.1, J15.3 (Pin_3), J16.3 (Pin_3); no longer U3.1 (A->B), U4.1 (A->B)
- net -12V: now also J15.4 (Pin_4), J16.4 (Pin_4)
- net -5V: now also J15.2 (Pin_2), J16.2 (Pin_2)
- net AD1: now also J2.1 (Pin_1)
- net AD10: now also J13.3 (Pin_3)
- net AD11: now also J13.4 (Pin_4)
- net AD12: now also J13.5 (Pin_5)
- net AD13: now also J13.6 (Pin_6)
- net AD14: now also J13.7 (Pin_7)
- net AD15: now also J13.8 (Pin_8)
- net AD2: now also J2.2 (Pin_2)
- net AD3: now also J2.3 (Pin_3)
- net AD4: now also J2.4 (Pin_4)
- net AD5: now also J2.5 (Pin_5)
- net AD6: now also J2.6 (Pin_6)
- net AD7: now also J2.7 (Pin_7)
- net AD8: now also J13.1 (Pin_1)
- net AD9: now also J13.2 (Pin_2)
- net BAD1: now also J6.1 (Pin_1)
- net BAD10: now also J14.3 (Pin_3)
- net BAD11: now also J14.4 (Pin_4)
- net BAD12: now also J14.5 (Pin_5)
- net BAD13: now also J14.6 (Pin_6)
- net BAD14: now also J14.7 (Pin_7)
- net BAD15: now also J14.8 (Pin_8)
- net BAD2: now also J6.2 (Pin_2)
- net BAD3: now also J6.3 (Pin_3)
- net BAD4: now also J6.4 (Pin_4)
- net BAD5: now also J6.5 (Pin_5)
- net BAD6: now also J6.6 (Pin_6)
- net BAD7: now also J6.7 (Pin_7)
- net BAD8: now also J14.1 (Pin_1)
- net BAD9: now also J14.2 (Pin_2)
- net GND: now also U3.1 (A->B), U4.1 (A->B), C1.2, C2.2, J15.5 (Pin_5), J16.5 (Pin_5)
Other:
- note added: "INSTALL BETWEEN CPU/ROM AND RAM BACKPLANES"
- moved on the sheet: J1, J11, J3, J4, J5, J7, J8, J9, U3, U4
