File: KiCad FIles/TMSHB_UART_ALL_V3/TMSHB_UART_ALL_V3.kicad_pcb (KiCad board)
At the start: 2 copper layers, 309.9 x 203.2 mm, 113 parts, among them J1 Conn_01x08_Pin, J10 Conn_01x02_Pin, J11 Conn_01x02_Pin, J12 Conn_01x02_Pin, J13 Conn_01x02_Pin, J14 Conn_01x02_Pin, J15 Conn_01x16_Pin, J16 Conn_01x08_Pin, J17 Conn_01x05_Pin, J18 Conn_01x05_Pin, J19 Conn_01x05_Pin, J2 Conn_01x15_Pin, J20 Conn_01x15_Pin, J21 Conn_01x15_Pin, J22 Conn_01x16_Pin, J23 Conn_01x08_Pin, J24 Conn_01x05_Pin, J25 Conn_01x05_Pin, J26 Conn_01x05_Pin, J27 Conn_01x12_Pin, J28 Conn_01x12_Pin, J29 Conn_01x12_Pin, J3 Conn_01x16_Pin, J30 Conn_01x02_Pin, J31 Conn_01x12_Pin, J32 Conn_01x02_Pin, J33 Conn_01x02_Pin, J34 Conn_01x02_Pin, J4 Conn_01x05_Pin, J5 Conn_01x05_Pin, J6 Conn_01x03_Pin, J7 Conn_01x05_Pin, J8 Conn_01x03_Pin, J9 Conn_01x02_Pin, Q1 NPN, Q13 NPN, Q14 PNP, Q2 PNP, Q3 NPN, Q4 NPN, U1 TR1602, U10 NE555P, U11 74LS138, U13 74LS138, U2 74LS04, U3 74LS00, U4 74LS32, U5 NE555P, U6 74LS00, U7 TR1602, U8 74LS00, U9 74LS32

Commit message: 2026/3/5
Parts:
- removed D10, D13, D14, D15, D16, D17, D7, D8, D9: D_Schottky, Diode_THT:D_DO-34_SOD68_P7.62mm_Horizontal
- removed J31: Conn_01x12_Pin, Connector_PinHeader_2.54mm:PinHeader_1x12_P2.54mm_Vertical
- removed J33: Conn_01x02_Pin, Connector_PinHeader_2.54mm:PinHeader_1x02_P2.54mm_Vertical
- added C18: C, Capacitor_THT:C_Disc_D3.0mm_W1.6mm_P2.50mm, F.Cu at (332.7, 141.0)
- added C22: C, Capacitor_THT:C_Disc_D3.0mm_W1.6mm_P2.50mm, F.Cu at (332.7, 144.2)
- added C23: 0.1u, Capacitor_THT:C_Disc_D3.0mm_W1.6mm_P2.50mm, F.Cu at (332.7, 147.3)
- added C24: 0.1u, Capacitor_THT:C_Disc_D3.0mm_W1.6mm_P2.50mm, F.Cu at (332.7, 150.5)
- added J35: Conn_01x14_Pin, Connector_PinHeader_2.54mm:PinHeader_1x14_P2.54mm_Vertical, F.Cu at (292.1, 106.7)
- added R14: 33k, Resistor_THT:R_Axial_DIN0207_L6.3mm_D2.5mm_P10.16mm_Horizontal, F.Cu at (370.8, 142.2)
- added R15: 33k, Resistor_THT:R_Axial_DIN0207_L6.3mm_D2.5mm_P10.16mm_Horizontal, F.Cu at (370.8, 146.3)
- added U12: 74LS148, Package_DIP:DIP-16_W7.62mm, F.Cu at (362.1, 97.0)
- added U14: 74LS00, Package_DIP:DIP-14_W7.62mm, F.Cu at (357.5, 119.4)
- added U15: NE555P, Package_DIP:DIP-8_W7.62mm, F.Cu at (368.3, 119.4)
- J10, J11, J12: value Conn_01x02_Pin -> Conn_01x14_Pin; footprint Connector_PinHeader_2.54mm:PinHeader_1x02_P2.54mm_Vertical -> Connector_PinHeader_2.54mm:PinHeader_1x14_P2.54mm_Vertical
- J13: value Conn_01x02_Pin -> Conn_01x15_Pin; footprint Connector_PinHeader_2.54mm:PinHeader_1x02_P2.54mm_Vertical -> Connector_PinHeader_2.54mm:PinHeader_1x15_P2.54mm_Vertical
- J14: value Conn_01x02_Pin -> Conn_01x16_Pin; footprint Connector_PinHeader_2.54mm:PinHeader_1x02_P2.54mm_Vertical -> Connector_PinHeader_2.54mm:PinHeader_1x16_P2.54mm_Vertical
- J27: value Conn_01x12_Pin -> Conn_01x08_Pin; footprint Connector_PinHeader_2.54mm:PinHeader_1x12_P2.54mm_Vertical -> Connector_PinHeader_2.54mm:PinHeader_1x08_P2.54mm_Vertical
- J28, J29: value Conn_01x12_Pin -> Conn_01x05_Pin; footprint Connector_PinHeader_2.54mm:PinHeader_1x12_P2.54mm_Vertical -> Connector_PinHeader_2.54mm:PinHeader_1x05_P2.54mm_Vertical
- J30: value Conn_01x02_Pin -> Conn_01x05_Pin; footprint Connector_PinHeader_2.54mm:PinHeader_1x02_P2.54mm_Vertical -> Connector_PinHeader_2.54mm:PinHeader_1x05_P2.54mm_Vertical
- J9: value Conn_01x02_Pin -> Interconnect; footprint Connector_PinHeader_2.54mm:PinHeader_1x02_P2.54mm_Vertical -> Connector_PinHeader_2.54mm:PinHeader_1x14_P2.54mm_Vertical
- moved J27 344.0 mm to (434.3, 142.2)
- moved J28 332.4 mm to (415.0, 142.2)
- moved J30 275.4 mm to (424.2, 142.2), turned to 0 degrees
- moved D6 242.6 mm to (373.4, 152.4)
- moved J9 188.7 mm to (91.4, 114.3), turned to 0 degrees
- moved J12 186.3 mm to (251.5, 114.3), turned to 0 degrees
- moved J29 184.6 mm to (419.6, 142.2)
- moved J14 180.4 mm to (447.4, 132.3), turned to 0 degrees
- moved J13 177.5 mm to (439.8, 132.3), turned to 0 degrees
- moved J10 107.8 mm to (91.4, 218.4), turned to 0 degrees
- moved J11 95.6 mm to (251.5, 218.4), turned to 0 degrees
Connections:
- D6 pad 1: Net-(D10-K) -> Net-(D6-K)
- D6 pad 2: Net-(D6-A) -> DA0_1
- J10 pad 1: IC1_0 -> M0STAT
- J10 pad 2: Net-(D7-A) -> M0RERD
- J11 pad 1: IC0_0 -> unconnected-(J11-Pin_1-Pad1)
- J11 pad 2: Net-(D6-A) -> unconnected-(J11-Pin_2-Pad2)
- J12 pad 1: IC0_1 -> unconnected-(J12-Pin_1-Pad1)
- J12 pad 2: Net-(D13-A) -> unconnected-(J12-Pin_2-Pad2)
- J13 pad 1: IC1_1 -> AD1_3
- J13 pad 2: Net-(D14-A) -> AD2_3
- J14 pad 1: IC2_1 -> DA0_1
- J14 pad 2: Net-(D15-A) -> DA1_1
- J17 pad 1: IRQ_1 -> unconnected-(J17-Pin_1-Pad1)
- J17 pad 2: IC0_1 -> unconnected-(J17-Pin_2-Pad2)
- J17 pad 3: IC1_1 -> unconnected-(J17-Pin_3-Pad3)
- J17 pad 4: IC2_1 -> unconnected-(J17-Pin_4-Pad4)
- J17 pad 5: IC3_1 -> unconnected-(J17-Pin_5-Pad5)
- J27 pad 1: Net-(J27-Pin_1) -> /DBIN
- J27 pad 2: Net-(J27-Pin_2) -> //MEMIN
- J27 pad 3: Net-(J27-Pin_3) -> /READY
- J27 pad 4: Net-(J27-Pin_4) -> //WE
- J27 pad 5: Net-(J27-Pin_5) -> //HOLD
- J27 pad 6: Net-(J27-Pin_6) -> /WAIT
- J27 pad 7: Net-(J27-Pin_7) -> /HOLDA
- J27 pad 8: Net-(J27-Pin_8) -> //RESET
- J28 pad 1: M0STAT -> IRQ_0
- J28 pad 2: M0RERD -> IC0_0
- J28 pad 3: /M0THL -> IC1_0
- J28 pad 4: /M0IQR -> IC2_0
- J28 pad 5: unconnected-(J28-Pin_5-Pad5) -> IC3_0
- J29 pad 5: M1STAT -> unconnected-(J29-Pin_5-Pad5)
- J30 pad 1: IC3_0 -> +12V
- J30 pad 2: Net-(D9-A) -> -5V
- J4 pad 1: IRQ_0 -> unconnected-(J4-Pin_1-Pad1)
- J4 pad 2: IC0_0 -> unconnected-(J4-Pin_2-Pad2)
- J4 pad 3: IC1_0 -> unconnected-(J4-Pin_3-Pad3)
- J4 pad 4: IC2_0 -> unconnected-(J4-Pin_4-Pad4)
- J4 pad 5: IC3_0 -> unconnected-(J4-Pin_5-Pad5)
- J9 pad 1: IC2_0 -> Net-(J9-Pin_1)
- J9 pad 2: Net-(D8-A) -> Net-(J9-Pin_2)
- U11 pad 12: Net-(J27-Pin_4) -> Net-(J9-Pin_4)
- U11 pad 13: Net-(J27-Pin_3) -> Net-(J9-Pin_3)
- U11 pad 7: Net-(J27-Pin_8) -> Net-(J9-Pin_8)
- U11 pad 9: Net-(J27-Pin_7) -> Net-(J9-Pin_7)
- U13 pad 12: Net-(J27-Pin_12) -> Net-(J9-Pin_12)
- U13 pad 13: Net-(J27-Pin_11) -> Net-(U13-O2)
- U13 pad 14: Net-(J27-Pin_10) -> Net-(J9-Pin_10)
- U13 pad 15: Net-(J27-Pin_9) -> Net-(J9-Pin_9)
- U2 pad 10: Net-(J27-Pin_2) -> Net-(J9-Pin_2)
- U2 pad 2: Net-(J27-Pin_5) -> Net-(J9-Pin_5)
- U2 pad 4: Net-(J27-Pin_6) -> Net-(J9-Pin_6)
- U2 pad 5: GND -> Net-(U13-O2)
- U2 pad 6: unconnected-(U2-Pad6) -> Net-(J9-Pin_11)
- U2 pad 8: Net-(J27-Pin_1) -> Net-(J9-Pin_1)
- U6 pad 11: Net-(D10-K) -> /PEN_0
- U6 pad 13: /M0IQR -> /M0RST
- U6 pad 5: Net-(D10-K) -> /PEN_0
- U8 pad 11: Net-(D13-K) -> /PEN_1
- U8 pad 13: /M1IQR -> /M1RST
- U8 pad 5: Net-(D13-K) -> /PEN_1
Routing:
- net Net-(J9-Pin_4): track 0.00 -> 108.3 mm, vias 0 -> 3
- net Net-(J27-Pin_4): track 108.3 -> 0.00 mm, vias 3 -> 0
- net Net-(J9-Pin_7): track 0.00 -> 107.1 mm, vias 0 -> 3
- net Net-(J27-Pin_7): track 107.1 -> 0.00 mm, vias 3 -> 0
- net Net-(J9-Pin_3): track 0.00 -> 99.4 mm, vias 0 -> 1
- net Net-(J27-Pin_3): track 99.4 -> 0.00 mm, vias 1 -> 0
- net Net-(J27-Pin_12): track 97.1 -> 0.00 mm, vias 3 -> 0
- net Net-(J9-Pin_8): track 0.00 -> 95.6 mm, vias 0 -> 3
- net Net-(J27-Pin_8): track 95.6 -> 0.00 mm, vias 3 -> 0
- net Net-(J27-Pin_11): track 89.4 -> 0.00 mm, vias 3 -> 0
- net Net-(J9-Pin_12): track 0.00 -> 89.4 mm, vias 0 -> 3
- net (no net): track 0.00 -> 87.3 mm
- net Net-(U13-O2): track 0.00 -> 79.1 mm, vias 0 -> 2
- net Net-(J9-Pin_9): track 0.00 -> 77.7 mm, vias 0 -> 3
- net Net-(J27-Pin_9): track 77.7 -> 0.00 mm, vias 3 -> 0
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
Commit message: 2026/4/6
Parts:
- moved J30 176.9 mm to (251.5, 180.3), turned to 90 degrees
- moved J13 169.8 mm to (276.9, 180.3), turned to 90 degrees
- moved J29 160.0 mm to (264.2, 180.3), turned to 90 degrees
- moved J15 160.0 mm to (348.0, 284.5)
- moved J3 160.0 mm to (188.0, 284.5)
- moved J27 125.3 mm to (315.0, 180.3), turned to 90 degrees
- moved J14 110.4 mm to (348.0, 180.3), turned to 90 degrees
- moved J28 88.4 mm to (335.3, 180.3), turned to 90 degrees
- moved U14 83.6 mm to (284.5, 160.0), turned to 90 degrees
- moved U15 82.3 mm to (287.0, 132.1), turned to 90 degrees
- moved R15 81.8 mm to (289.6, 137.2), turned to 180 degrees
- moved R14 81.3 mm to (289.6, 139.7), turned to 180 degrees
- moved U12 78.7 mm to (315.0, 160.0), turned to 90 degrees
- moved D6 65.0 mm to (308.6, 147.3)
- moved C22 54.4 mm to (279.4, 154.9), turned to -90 degrees
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Connections:
- D19 pad 2: DA0_1 -> DA0_2
- D20 pad 2: DA1_1 -> DA1_2
- D6 pad 2: DA0_1 -> DA0_3
- J13 pad 1: AD1_3 -> unconnected-(J13-Pin_1-Pad1)
- J13 pad 10: AD10_3 -> unconnected-(J13-Pin_10-Pad10)
- J13 pad 11: AD11_3 -> unconnected-(J13-Pin_11-Pad11)
- J13 pad 12: AD12_3 -> unconnected-(J13-Pin_12-Pad12)
- J13 pad 13: AD13_3 -> unconnected-(J13-Pin_13-Pad13)
- J13 pad 14: AD14_3 -> unconnected-(J13-Pin_14-Pad14)
- J13 pad 15: AD15_3 -> unconnected-(J13-Pin_15-Pad15)
- J13 pad 2: AD2_3 -> unconnected-(J13-Pin_2-Pad2)
- J13 pad 3: AD3_3 -> unconnected-(J13-Pin_3-Pad3)
- J13 pad 4: AD4_3 -> unconnected-(J13-Pin_4-Pad4)
- J13 pad 5: AD5_3 -> unconnected-(J13-Pin_5-Pad5)
- J13 pad 6: AD6_3 -> unconnected-(J13-Pin_6-Pad6)
- J13 pad 7: AD7_3 -> unconnected-(J13-Pin_7-Pad7)
- J13 pad 8: AD8_3 -> unconnected-(J13-Pin_8-Pad8)
- J13 pad 9: AD9_3 -> unconnected-(J13-Pin_9-Pad9)
- J14 pad 1: DA0_1 -> DA0_3
- J14 pad 10: /DA9 -> unconnected-(J14-Pin_10-Pad10)
- J14 pad 11: /DA10 -> unconnected-(J14-Pin_11-Pad11)
- J14 pad 12: /DA11 -> unconnected-(J14-Pin_12-Pad12)
- J14 pad 13: /DA12 -> unconnected-(J14-Pin_13-Pad13)
- J14 pad 14: /DA13 -> unconnected-(J14-Pin_14-Pad14)
- J14 pad 15: /DA14 -> unconnected-(J14-Pin_15-Pad15)
- J14 pad 16: /DA15 -> unconnected-(J14-Pin_16-Pad16)
- J14 pad 2: DA1_1 -> DA1_3
- J14 pad 3: DA2_1 -> DA2_3
- J14 pad 4: DA3_1 -> DA3_3
- J14 pad 5: DA4_1 -> DA4_3
- J14 pad 6: DA5_1 -> DA5_3
- J14 pad 7: DA6_1 -> DA6_3
- J14 pad 8: DA7_1 -> unconnected-(J14-Pin_8-Pad8)
- J14 pad 9: /DA8 -> unconnected-(J14-Pin_9-Pad9)
- J15 pad 1: DA0_1 -> DA0_2
- J15 pad 10: /DA9 -> unconnected-(J15-Pin_10-Pad10)
- J15 pad 11: /DA10 -> unconnected-(J15-Pin_11-Pad11)
- J15 pad 12: /DA11 -> unconnected-(J15-Pin_12-Pad12)
- J15 pad 13: /DA12 -> unconnected-(J15-Pin_13-Pad13)
- J15 pad 14: /DA13 -> unconnected-(J15-Pin_14-Pad14)
- J15 pad 15: /DA14 -> unconnected-(J15-Pin_15-Pad15)
- J15 pad 16: /DA15 -> unconnected-(J15-Pin_16-Pad16)
- J15 pad 2: DA1_1 -> DA1_2
- J15 pad 3: DA2_1 -> DA2_2
- J15 pad 4: DA3_1 -> DA3_2
- J15 pad 5: DA4_1 -> DA4_2
- J15 pad 6: DA5_1 -> DA5_2
- J15 pad 7: DA6_1 -> DA6_2
- J15 pad 8: DA7_1 -> DA7_2
- J15 pad 9: /DA8 -> unconnected-(J15-Pin_9-Pad9)
- J16 pad 1: /DBIN -> unconnected-(J16-Pin_1-Pad1)
- J16 pad 2: //MEMIN -> unconnected-(J16-Pin_2-Pad2)
- J16 pad 3: /READY -> unconnected-(J16-Pin_3-Pad3)
- J16 pad 4: //WE -> unconnected-(J16-Pin_4-Pad4)
- J16 pad 5: //HOLD -> unconnected-(J16-Pin_5-Pad5)
- J16 pad 6: /WAIT -> unconnected-(J16-Pin_6-Pad6)
- J16 pad 7: /HOLDA -> unconnected-(J16-Pin_7-Pad7)
- J16 pad 8: //RESET -> unconnected-(J16-Pin_8-Pad8)
- J2 pad 1: AD1_3 -> /AD1
- J2 pad 10: AD10_3 -> /AD10
- J2 pad 11: AD11_3 -> /AD11
- J2 pad 12: AD12_3 -> /AD12
- J2 pad 13: AD13_3 -> /AD13
- J2 pad 14: AD14_3 -> /AD14
- J2 pad 15: AD15_3 -> /AD15
- J2 pad 2: AD2_3 -> /AD2
- J2 pad 3: AD3_3 -> /AD3
- J2 pad 4: AD4_3 -> /AD4
- J2 pad 5: AD5_3 -> /AD5
- J2 pad 6: AD6_3 -> /AD6
- J2 pad 7: AD7_3 -> /AD7
- J2 pad 8: AD8_3 -> /AD8
- J2 pad 9: AD9_3 -> /AD9
- J20 pad 1: AD1_3 -> unconnected-(J20-Pin_1-Pad1)
- J20 pad 10: AD10_3 -> unconnected-(J20-Pin_10-Pad10)
- J20 pad 11: AD11_3 -> unconnected-(J20-Pin_11-Pad11)
- J20 pad 12: AD12_3 -> unconnected-(J20-Pin_12-Pad12)
- J20 pad 13: AD13_3 -> unconnected-(J20-Pin_13-Pad13)
- J20 pad 14: AD14_3 -> unconnected-(J20-Pin_14-Pad14)
- J20 pad 15: AD15_3 -> unconnected-(J20-Pin_15-Pad15)
- J20 pad 2: AD2_3 -> unconnected-(J20-Pin_2-Pad2)
- J20 pad 3: AD3_3 -> unconnected-(J20-Pin_3-Pad3)
- J20 pad 4: AD4_3 -> unconnected-(J20-Pin_4-Pad4)
- J20 pad 5: AD5_3 -> unconnected-(J20-Pin_5-Pad5)
- J20 pad 6: AD6_3 -> unconnected-(J20-Pin_6-Pad6)
- J20 pad 7: AD7_3 -> unconnected-(J20-Pin_7-Pad7)
- J20 pad 8: AD8_3 -> unconnected-(J20-Pin_8-Pad8)
- J20 pad 9: AD9_3 -> unconnected-(J20-Pin_9-Pad9)
- J22 pad 1: DA0_1 -> unconnected-(J22-Pin_1-Pad1)
- J22 pad 10: /DA9 -> unconnected-(J22-Pin_10-Pad10)
- J22 pad 11: /DA10 -> unconnected-(J22-Pin_11-Pad11)
- J22 pad 12: /DA11 -> unconnected-(J22-Pin_12-Pad12)
- J22 pad 13: /DA12 -> unconnected-(J22-Pin_13-Pad13)
- J22 pad 14: /DA13 -> unconnected-(J22-Pin_14-Pad14)
- J22 pad 15: /DA14 -> unconnected-(J22-Pin_15-Pad15)
- J22 pad 16: /DA15 -> unconnected-(J22-Pin_16-Pad16)
- J22 pad 2: DA1_1 -> unconnected-(J22-Pin_2-Pad2)
- J22 pad 3: DA2_1 -> unconnected-(J22-Pin_3-Pad3)
- J22 pad 4: DA3_1 -> unconnected-(J22-Pin_4-Pad4)
- J22 pad 5: DA4_1 -> unconnected-(J22-Pin_5-Pad5)
- J22 pad 6: DA5_1 -> unconnected-(J22-Pin_6-Pad6)
- J22 pad 7: DA6_1 -> unconnected-(J22-Pin_7-Pad7)
- J22 pad 8: DA7_1 -> unconnected-(J22-Pin_8-Pad8)
- J22 pad 9: /DA8 -> unconnected-(J22-Pin_9-Pad9)
- J23 pad 1: /DBIN -> unconnected-(J23-Pin_1-Pad1)
- J23 pad 2: //MEMIN -> unconnected-(J23-Pin_2-Pad2)
- J23 pad 3: /READY -> unconnected-(J23-Pin_3-Pad3)
- J23 pad 4: //WE -> unconnected-(J23-Pin_4-Pad4)
- J23 pad 5: //HOLD -> unconnected-(J23-Pin_5-Pad5)
- J23 pad 6: /WAIT -> unconnected-(J23-Pin_6-Pad6)
- J23 pad 7: /HOLDA -> unconnected-(J23-Pin_7-Pad7)
- J23 pad 8: //RESET -> unconnected-(J23-Pin_8-Pad8)
- J27 pad 1: /DBIN -> unconnected-(J27-Pin_1-Pad1)
- J27 pad 2: //MEMIN -> unconnected-(J27-Pin_2-Pad2)
- J27 pad 3: /READY -> unconnected-(J27-Pin_3-Pad3)
- J27 pad 4: //WE -> unconnected-(J27-Pin_4-Pad4)
- J27 pad 5: //HOLD -> unconnected-(J27-Pin_5-Pad5)
- J27 pad 6: /WAIT -> unconnected-(J27-Pin_6-Pad6)
- J27 pad 7: /HOLDA -> unconnected-(J27-Pin_7-Pad7)
- J27 pad 8: //RESET -> unconnected-(J27-Pin_8-Pad8)
- J29 pad 1: unconnected-(J29-Pin_1-Pad1) -> /TAPE
- J35 pad 3: DA0_1 -> DA0_3
- J35 pad 4: DA1_1 -> DA1_3
- J35 pad 5: DA2_1 -> DA2_3
- J35 pad 6: DA3_1 -> DA3_3
- J35 pad 7: DA4_1 -> DA4_3
- J35 pad 8: DA5_1 -> DA5_3
- J35 pad 9: DA6_1 -> DA6_3
- U7 pad 10: DA2_1 -> DA2_2
- U7 pad 11: DA1_1 -> DA1_2
- U7 pad 12: DA0_1 -> DA0_2
- U7 pad 26: DA0_1 -> DA0_2
- U7 pad 27: DA1_1 -> DA1_2
- U7 pad 28: DA2_1 -> DA2_2
- U7 pad 29: DA3_1 -> DA3_2
- U7 pad 30: DA4_1 -> DA4_2
- U7 pad 31: DA5_1 -> DA5_2
- U7 pad 32: DA6_1 -> DA6_2
- U7 pad 33: DA7_1 -> DA7_2
- U7 pad 5: DA7_1 -> DA7_2
- U7 pad 6: DA6_1 -> DA6_2
- U7 pad 7: DA5_1 -> DA5_2
- U7 pad 8: DA4_1 -> DA4_2
- U7 pad 9: DA3_1 -> DA3_2
Routing:
- net GND: track 1239.6 -> 1605.5 mm, vias 41 -> 47
- net +5V: track 1300.4 -> 1533.2 mm, vias 33 -> 38
- net /PPRF: track 2.54 -> 168.0 mm, vias 1 -> 8
- net PSTRB: track 2.54 -> 142.4 mm, vias 1 -> 6
- net Net-(J35-Pin_12): track 0.00 -> 128.7 mm, vias 0 -> 3
- net /M0IQR: track 126.1 -> 0.00 mm, vias 5 -> 0
- net DA0_3: track 0.00 -> 125.9 mm, vias 0 -> 2
- net DA1_1: track 233.3 -> 115.4 mm, vias 3 -> 1
- net DA1_2: track 0.00 -> 115.4 mm, vias 0 -> 1
- net /M1IQR: track 112.2 -> 0.00 mm, vias 2 -> 0
- net /PEN_M0: track 0.00 -> 110.7 mm, vias 0 -> 3
- net /PEN_M1: track 0.00 -> 106.8 mm, vias 0 -> 3
- net DA0_1: track 207.6 -> 102.5 mm, vias 3 -> 1
- net DA0_2: track 0.00 -> 102.5 mm, vias 0 -> 1
- net DA7_1: track 193.0 -> 95.2 mm, vias 3 -> 1
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
Commit message: 2026/4/6
Parts:
- added C25: 1u, Capacitor_THT:C_Disc_D3.0mm_W1.6mm_P2.50mm, F.Cu at (160.0, 221.0)
- added C26: 1u, Capacitor_THT:C_Disc_D3.0mm_W1.6mm_P2.50mm, F.Cu at (320.0, 221.0)
- added D7: D, Diode_THT:D_DO-34_SOD68_P7.62mm_Horizontal, F.Cu at (152.4, 221.0)
- added D8: D, Diode_THT:D_DO-34_SOD68_P7.62mm_Horizontal, F.Cu at (312.4, 221.0)
- added Q5: NPN, Package_TO_SOT_THT:TO-92_Inline_Wide, F.Cu at (127.0, 248.9)
- added Q6: NPN, Package_TO_SOT_THT:TO-92_Inline_Wide, F.Cu at (287.0, 248.9)
- added R17: 1k, Resistor_THT:R_Axial_DIN0207_L6.3mm_D2.5mm_P10.16mm_Horizontal, F.Cu at (154.9, 210.8)
- added R18: 10k, Resistor_THT:R_Axial_DIN0207_L6.3mm_D2.5mm_P10.16mm_Horizontal, F.Cu at (106.7, 223.5)
- added R19: 4.7k, Resistor_THT:R_Axial_DIN0207_L6.3mm_D2.5mm_P10.16mm_Horizontal, F.Cu at (96.5, 254.0)
- added R20: 1k, Resistor_THT:R_Axial_DIN0207_L6.3mm_D2.5mm_P10.16mm_Horizontal, F.Cu at (315.0, 210.8)
- added R21: 10k, Resistor_THT:R_Axial_DIN0207_L6.3mm_D2.5mm_P10.16mm_Horizontal, F.Cu at (266.7, 231.1)
- added R27: 4.7k, Resistor_THT:R_Axial_DIN0207_L6.3mm_D2.5mm_P10.16mm_Horizontal, F.Cu at (256.5, 254.0)
- R14: value 33k -> 220k
- R15: value 33k -> 4.7k
- moved C4 21.8 mm to (221.0, 210.9), turned to -90 degrees
- moved C8 21.8 mm to (381.0, 210.9), turned to -90 degrees
- moved RV1 14.4 mm to (215.9, 213.4), turned to -90 degrees
- moved RV2 14.4 mm to (375.9, 213.4), turned to -90 degrees
- moved R4 10.5 mm to (210.8, 215.9), turned to 90 degrees
- moved R26 10.5 mm to (370.8, 215.9), turned to 90 degrees
- moved C5 3.56 mm to (208.2, 213.4), turned to 180 degrees
- moved C7 3.54 mm to (368.3, 213.4), turned to 180 degrees
- moved D6 2.54 mm to (308.6, 144.8)
Connections:
- D19 pad 2: DA0_2 -> DA8_2
- D20 pad 2: DA1_2 -> DA9_2
- D4 pad 2: DA0_1 -> DA8_1
- D5 pad 2: DA1_1 -> DA9_1
- J15 pad 1: DA0_2 -> unconnected-(J15-Pin_1-Pad1)
- J15 pad 10: unconnected-(J15-Pin_10-Pad10) -> DA9_2
- J15 pad 11: unconnected-(J15-Pin_11-Pad11) -> DA10_2
- J15 pad 12: unconnected-(J15-Pin_12-Pad12) -> DA11_2
- J15 pad 13: unconnected-(J15-Pin_13-Pad13) -> DA12_2
- J15 pad 14: unconnected-(J15-Pin_14-Pad14) -> DA13_2
- J15 pad 15: unconnected-(J15-Pin_15-Pad15) -> DA14_2
- J15 pad 16: unconnected-(J15-Pin_16-Pad16) -> DA15_2
- J15 pad 2: DA1_2 -> unconnected-(J15-Pin_2-Pad2)
- J15 pad 3: DA2_2 -> unconnected-(J15-Pin_3-Pad3)
- J15 pad 4: DA3_2 -> unconnected-(J15-Pin_4-Pad4)
- J15 pad 5: DA4_2 -> unconnected-(J15-Pin_5-Pad5)
- J15 pad 6: DA5_2 -> unconnected-(J15-Pin_6-Pad6)
- J15 pad 7: DA6_2 -> unconnected-(J15-Pin_7-Pad7)
- J15 pad 8: DA7_2 -> unconnected-(J15-Pin_8-Pad8)
- J15 pad 9: unconnected-(J15-Pin_9-Pad9) -> DA8_2
- J3 pad 1: DA0_1 -> /DA0
- J3 pad 10: /DA9 -> DA9_1
- J3 pad 11: /DA10 -> DA10_1
- J3 pad 12: /DA11 -> DA11_1
- J3 pad 13: /DA12 -> DA12_1
- J3 pad 14: /DA13 -> DA13_1
- J3 pad 15: /DA14 -> DA14_1
- J3 pad 16: /DA15 -> DA15_1
- J3 pad 2: DA1_1 -> /DA1
- J3 pad 3: DA2_1 -> /DA2
- J3 pad 4: DA3_1 -> /DA3
- J3 pad 5: DA4_1 -> /DA4
- J3 pad 6: DA5_1 -> /DA5
- J3 pad 7: DA6_1 -> /DA6
- J3 pad 8: DA7_1 -> /DA7
- J3 pad 9: /DA8 -> DA8_1
- U1 pad 10: DA2_1 -> DA10_1
- U1 pad 11: DA1_1 -> DA9_1
- U1 pad 12: DA0_1 -> DA8_1
- U1 pad 18: /M0IQR -> Net-(Q5-C)
- U1 pad 26: DA0_1 -> DA8_1
- U1 pad 27: DA1_1 -> DA9_1
- U1 pad 28: DA2_1 -> DA10_1
- U1 pad 29: DA3_1 -> DA11_1
- U1 pad 30: DA4_1 -> DA12_1
- U1 pad 31: DA5_1 -> DA13_1
- U1 pad 32: DA6_1 -> DA14_1
- U1 pad 33: DA7_1 -> DA15_1
- U1 pad 5: DA7_1 -> DA15_1
- U1 pad 6: DA6_1 -> DA14_1
- U1 pad 7: DA5_1 -> DA13_1
- U1 pad 8: DA4_1 -> DA12_1
- U1 pad 9: DA3_1 -> DA11_1
- U12 pad 1: /PEN_M1 -> /PEN_M0
- U12 pad 12: unconnected-(U12-I2-Pad12) -> Net-(U12-I2)
- U12 pad 13: Net-(U12-I3) -> /PEN_M1
- U12 pad 2: /PEN_M0 -> /TAPE
- U12 pad 3: /TAPE -> unconnected-(U12-I6-Pad3)
- U14 pad 2: Net-(U12-I3) -> Net-(U12-I2)
- U14 pad 6: Net-(U12-I3) -> Net-(U12-I2)
- U4 pad 12: Net-(U1-DR) -> Net-(D7-K)
- U7 pad 10: DA2_2 -> DA10_2
- U7 pad 11: DA1_2 -> DA9_2
- U7 pad 12: DA0_2 -> DA8_2
- U7 pad 18: /M1IQR -> Net-(Q6-C)
- U7 pad 26: DA0_2 -> DA8_2
- U7 pad 27: DA1_2 -> DA9_2
- U7 pad 28: DA2_2 -> DA10_2
- U7 pad 29: DA3_2 -> DA11_2
- U7 pad 30: DA4_2 -> DA12_2
- U7 pad 31: DA5_2 -> DA13_2
- U7 pad 32: DA6_2 -> DA14_2
- U7 pad 33: DA7_2 -> DA15_2
- U7 pad 5: DA7_2 -> DA15_2
- U7 pad 6: DA6_2 -> DA14_2
- U7 pad 7: DA5_2 -> DA13_2
- U7 pad 8: DA4_2 -> DA12_2
- U7 pad 9: DA3_2 -> DA11_2
- U9 pad 12: Net-(U7-DR) -> Net-(D8-K)
Routing:
- net DA9_2: track 0.00 -> 135.7 mm, vias 0 -> 1
- net DA9_1: track 0.00 -> 135.7 mm, vias 0 -> 1
- net DA8_2: track 0.00 -> 122.8 mm, vias 0 -> 1
- net DA8_1: track 0.00 -> 122.8 mm, vias 0 -> 1
- net DA15_1: track 0.00 -> 115.5 mm, vias 0 -> 1
- net DA15_2: track 0.00 -> 115.5 mm, vias 0 -> 1
- net DA1_2: track 115.4 -> 0.00 mm, vias 1 -> 0
- net DA1_1: track 115.4 -> 0.00 mm, vias 1 -> 0
- net DA14_1: track 0.00 -> 111.7 mm, vias 0 -> 1
- net DA14_2: track 0.00 -> 111.7 mm, vias 0 -> 1
- net GND: track 1605.5 -> 1716.4 mm, vias 47 -> 51
- net DA13_1: track 0.00 -> 107.8 mm, vias 0 -> 1
- net DA13_2: track 0.00 -> 107.8 mm, vias 0 -> 1
- net DA12_1: track 0.00 -> 103.9 mm, vias 0 -> 1
- net DA12_2: track 0.00 -> 103.9 mm, vias 0 -> 1
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
Commit message: 2026/4/7
Parts:
- added J31: Conn_01x14_Pin, Connector_PinHeader_2.54mm:PinHeader_1x14_P2.54mm_Vertical, F.Cu at (198.1, 315.0)
- added J33: Conn_01x14_Pin, Connector_PinHeader_2.54mm:PinHeader_1x14_P2.54mm_Vertical, F.Cu at (215.9, 315.0)
- added J36: Conn_01x14_Pin, Connector_PinHeader_2.54mm:PinHeader_1x14_P2.54mm_Vertical, F.Cu at (233.7, 315.0)
- added J37: Conn_01x14_Pin, Connector_PinHeader_2.54mm:PinHeader_1x14_P2.54mm_Vertical, F.Cu at (251.5, 315.0)
Connections:
- D6 pad 2: DA0_3 -> DA8_3
- J14 pad 1: DA0_3 -> unconnected-(J14-Pin_1-Pad1)
- J14 pad 10: unconnected-(J14-Pin_10-Pad10) -> DA9_3
- J14 pad 11: unconnected-(J14-Pin_11-Pad11) -> DA10_3
- J14 pad 12: unconnected-(J14-Pin_12-Pad12) -> DA11_3
- J14 pad 13: unconnected-(J14-Pin_13-Pad13) -> DA12_3
- J14 pad 14: unconnected-(J14-Pin_14-Pad14) -> DA13_3
- J14 pad 15: unconnected-(J14-Pin_15-Pad15) -> DA14_3
- J14 pad 2: DA1_3 -> unconnected-(J14-Pin_2-Pad2)
- J14 pad 3: DA2_3 -> unconnected-(J14-Pin_3-Pad3)
- J14 pad 4: DA3_3 -> unconnected-(J14-Pin_4-Pad4)
- J14 pad 5: DA4_3 -> unconnected-(J14-Pin_5-Pad5)
- J14 pad 6: DA5_3 -> unconnected-(J14-Pin_6-Pad6)
- J14 pad 7: DA6_3 -> unconnected-(J14-Pin_7-Pad7)
- J14 pad 9: unconnected-(J14-Pin_9-Pad9) -> DA8_3
- J35 pad 3: DA0_3 -> DA8_3
- J35 pad 4: DA1_3 -> DA9_3
- J35 pad 5: DA2_3 -> DA10_3
- J35 pad 6: DA3_3 -> DA11_3
- J35 pad 7: DA4_3 -> DA12_3
- J35 pad 8: DA5_3 -> DA13_3
- J35 pad 9: DA6_3 -> DA14_3
Routing:
- net DA8_3: track 0.00 -> 169.7 mm, vias 0 -> 2
- net DA0_3: track 125.9 -> 0.00 mm, vias 2 -> 0
- net DA14_3: track 0.00 -> 99.7 mm, vias 0 -> 2
- net DA10_3: track 0.00 -> 99.7 mm, vias 0 -> 2
- net DA12_3: track 0.00 -> 99.7 mm, vias 0 -> 2
- net DA11_3: track 0.00 -> 99.7 mm, vias 0 -> 2
- net DA13_3: track 0.00 -> 99.7 mm, vias 0 -> 2
- net DA9_3: track 0.00 -> 99.7 mm, vias 0 -> 2
- net DA6_3: track 88.9 -> 0.00 mm, vias 2 -> 0
- net DA5_3: track 88.9 -> 0.00 mm, vias 2 -> 0
- net DA4_3: track 88.9 -> 0.00 mm, vias 2 -> 0
- net DA3_3: track 88.9 -> 0.00 mm, vias 2 -> 0
- net DA2_3: track 88.9 -> 0.00 mm, vias 2 -> 0
- net DA1_3: track 88.9 -> 0.00 mm, vias 2 -> 0
- net Net-(J31-Pin_9): track 0.00 -> 55.9 mm, vias 0 -> 4
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Other:
- board size 309.9 x 203.2 mm -> 309.9 x 264.2 mm

Commit message: 2026/4/9
Routing:
- net +5V: track 1548.6 -> 1551.2 mm
Changed lines of the file:
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@@
 	)
 	(segment
+		(start 256.54 256.54)
+		(end 256.54 254)
+		(width 1)
+		(layer "B.Cu")
+		(net 1)
+	)
+	(segment
 		(start 261.62 198.12)
 		(end 276.86 198.12)
@@
 	)
 	(segment
-		(start 254 213.36)
-		(end 251.46 213.36)
-		(width 1)
-		(layer "B.Cu")
-		(net 2)
-	)
-	(segment
 		(start 101.6 287.02)
 		(end 101.6 284.48)
@@
 	)
 	(segment
+		(start 251.46 213.36)
+		(end 254 213.36)
+		(width 1)
+		(layer "B.Cu")
+		(net 2)
+	)
+	(segment
 		(start 195.54 215.86)
 		(end 182.92 215.86)
@@
 	)
 	(arc
-		(start 251.46 213.36)
-		(mid 249.663949 212.616051)
-		(end 248.92 210.82)
-		(width 1)
-		(layer "B.Cu")
-		(net 2)
-	)
-	(arc
 		(start 322.58 266.7)
 		(mid 321.836051 268.496051)
@@
 		(width 1)
 		(layer "B.Cu")
+		(net 2)
+	)
+	(arc
+		(start 248.92 210.82)
+		(mid 249.663949 212.616051)
+		(end 251.46 213.36)
+		(width 1)
+		(layer "B.Cu")

Commit message: 2026/6/10
Parts:
- removed D11, D12: D_Schottky, Diode_THT:D_DO-34_SOD68_P7.62mm_Horizontal
- added Q7: NPN, Package_TO_SOT_THT:TO-92_Inline_Wide, F.Cu at (182.9, 147.3)
- added Q8: NPN, Package_TO_SOT_THT:TO-92_Inline_Wide, F.Cu at (190.5, 147.3)
- added R28: 10k, Resistor_THT:R_Axial_DIN0207_L6.3mm_D2.5mm_P10.16mm_Horizontal, F.Cu at (182.9, 134.6)
- added R29: 10k, Resistor_THT:R_Axial_DIN0207_L6.3mm_D2.5mm_P10.16mm_Horizontal, F.Cu at (193.0, 142.2)
- C4: value 470nF -> 47nF
Routing:
- net +5V: track 1551.2 -> 1592.1 mm
- net Net-(Q7-B): track 0.00 -> 17.9 mm
- net Net-(R28-Pad2): track 2.54 -> 19.1 mm
- net Net-(Q7-E): track 119.7 -> 131.4 mm, vias 8 -> 6
- net Net-(Q8-B): track 0.00 -> 8.97 mm
- net Net-(R29-Pad2): track 2.54 -> 5.08 mm
