File: KiCad FIles/TMSHB_UART_ALL_V3/TMSHB_UART_ALL_V3.kicad_sch (KiCad schematic)
At the start: 113 parts, among them J1 Conn_01x08_Pin, J10 Conn_01x14_Pin, J11 Conn_01x14_Pin, J12 Conn_01x14_Pin, J13 Conn_01x15_Pin, J14 Conn_01x16_Pin, J15 Conn_01x16_Pin, J16 Conn_01x08_Pin, J17 Conn_01x05_Pin, J18 Conn_01x05_Pin, J19 Conn_01x05_Pin, J2 Conn_01x15_Pin, J20 Conn_01x15_Pin, J21 Conn_01x15_Pin, J22 Conn_01x16_Pin, J23 Conn_01x08_Pin, J24 Conn_01x05_Pin, J25 Conn_01x05_Pin, J26 Conn_01x05_Pin, J27 Conn_01x08_Pin, J28 Conn_01x05_Pin, J29 Conn_01x05_Pin, J3 Conn_01x16_Pin, J30 Conn_01x05_Pin, J32 Conn_01x02_Pin, J34 Conn_01x02_Pin, J35 Conn_01x14_Pin, J4 Conn_01x05_Pin, J5 Conn_01x05_Pin, J6 Conn_01x03_Pin, J7 Conn_01x05_Pin, J8 Conn_01x03_Pin, J9 Interconnect, Q1 NPN, Q13 NPN, Q14 PNP, Q2 PNP, Q3 NPN, Q4 NPN, U1 TR1602, U10 NE555P, U11 74LS138, U12 74LS148, U13 74LS138, U14 74LS00, U15 NE555P, U16 74LS00, U2 74LS04, U3 74LS00, U4 74LS32, U5 NE555P, U6 74LS00, U7 TR1602, U8 74LS00, U9 74LS32

Commit message: 2026/3/5
Parts:
- removed U16: 74LS00, symbol 74xx:74LS00
- J10, J11, J12, J35, J9: footprint (none) -> Connector_PinHeader_2.54mm:PinHeader_1x14_P2.54mm_Vertical
- U12: footprint (none) -> Package_DIP:DIP-16_W7.62mm
- U14: footprint (none) -> Package_DIP:DIP-14_W7.62mm
Connections:
- net /PPORT is gone; now on an unnamed net: U12.13 (I3)
- net GND: now also U14.12, U14.13
- net PBUSY: now also U14.9
- net /PEN_M0: now also U12.2 (I5); no longer U12.11 (I1)
- net /PEN_M1: now also U12.1 (I4); no longer U12.12 (I2)
- net /TAPE: now also U12.3 (I6); no longer U12.10 (IO)
- net at D6.1 (K): now also U14.8
- net at J35.12 (Pin_12): now also U14.10
- net at U14.2, U14.6: no longer U12.1 (I4)
Other:
- moved on the sheet: J35, U12, U14A, U14B, U14C, U14D, U15

Commit message: 2026/4/6
Connections:
- net AD10_3: no longer J13.10 (Pin_10), J2.10 (Pin_10), J20.10 (Pin_10)
- net AD11_3: no longer J13.11 (Pin_11), J2.11 (Pin_11), J20.11 (Pin_11)
- net AD12_3: no longer J13.12 (Pin_12), J2.12 (Pin_12), J20.12 (Pin_12)
- net AD13_3: no longer J13.13 (Pin_13), J2.13 (Pin_13), J20.13 (Pin_13)
- net AD14_3: no longer J13.14 (Pin_14), J2.14 (Pin_14), J20.14 (Pin_14)
- net AD15_3: no longer J13.15 (Pin_15), J2.15 (Pin_15), J20.15 (Pin_15)
- net AD1_3: no longer J13.1 (Pin_1), J2.1 (Pin_1), J20.1 (Pin_1)
- net AD2_3: no longer J13.2 (Pin_2), J2.2 (Pin_2), J20.2 (Pin_2)
- net AD3_3: no longer J13.3 (Pin_3), J2.3 (Pin_3), J20.3 (Pin_3)
- net AD4_3: no longer J13.4 (Pin_4), J2.4 (Pin_4), J20.4 (Pin_4)
- net AD5_3: no longer J13.5 (Pin_5), J2.5 (Pin_5), J20.5 (Pin_5)
- net AD6_3: no longer J13.6 (Pin_6), J2.6 (Pin_6), J20.6 (Pin_6)
- net AD7_3: no longer J13.7 (Pin_7), J2.7 (Pin_7), J20.7 (Pin_7)
- net AD8_3: no longer J13.8 (Pin_8), J2.8 (Pin_8), J20.8 (Pin_8)
- net AD9_3: no longer J13.9 (Pin_9), J2.9 (Pin_9), J20.9 (Pin_9)
- net DA0_1: no longer D19.2 (A), D6.2 (A), J14.1 (Pin_1), J15.1 (Pin_1), J22.1 (Pin_1), J35.3 (Pin_3), U7.12 (RR1), U7.26 (TR1)
- net DA10: no longer J14.11 (Pin_11), J15.11 (Pin_11), J22.11 (Pin_11)
- net DA11: no longer J14.12 (Pin_12), J15.12 (Pin_12), J22.12 (Pin_12)
- net DA12: no longer J14.13 (Pin_13), J15.13 (Pin_13), J22.13 (Pin_13)
- net DA13: no longer J14.14 (Pin_14), J15.14 (Pin_14), J22.14 (Pin_14)
- net DA14: no longer J14.15 (Pin_15), J15.15 (Pin_15), J22.15 (Pin_15)
- net DA15: no longer J14.16 (Pin_16), J15.16 (Pin_16), J22.16 (Pin_16)
- net DA1_1: no longer D20.2 (A), J14.2 (Pin_2), J15.2 (Pin_2), J22.2 (Pin_2), J35.4 (Pin_4), U7.11 (RR2), U7.27 (TR2)
- net DA2_1: no longer J14.3 (Pin_3), J15.3 (Pin_3), J22.3 (Pin_3), J35.5 (Pin_5), U7.10 (RR3), U7.28 (TR3)
- net DA3_1: no longer J14.4 (Pin_4), J15.4 (Pin_4), J22.4 (Pin_4), J35.6 (Pin_6), U7.29 (TR4), U7.9 (RR4)
- net DA4_1: no longer J14.5 (Pin_5), J15.5 (Pin_5), J22.5 (Pin_5), J35.7 (Pin_7), U7.30 (TR5), U7.8 (RR5)
- net DA5_1: no longer J14.6 (Pin_6), J15.6 (Pin_6), J22.6 (Pin_6), J35.8 (Pin_8), U7.31 (TR6), U7.7 (RR6)
- net DA6_1: no longer J14.7 (Pin_7), J15.7 (Pin_7), J22.7 (Pin_7), J35.9 (Pin_9), U7.32 (TR7), U7.6 (RR7)
- net DA7_1: no longer J14.8 (Pin_8), J15.8 (Pin_8), J22.8 (Pin_8), U7.33 (TR8), U7.5 (RR8)
- net DA8: no longer J14.9 (Pin_9), J15.9 (Pin_9), J22.9 (Pin_9)
- net DA9: no longer J14.10 (Pin_10), J15.10 (Pin_10), J22.10 (Pin_10)
- net DBIN: no longer J16.1 (Pin_1), J23.1 (Pin_1), J27.1 (Pin_1)
- net HOLDA: no longer J16.7 (Pin_7), J23.7 (Pin_7), J27.7 (Pin_7)
- net READY: no longer J16.3 (Pin_3), J23.3 (Pin_3), J27.3 (Pin_3)
- net WAIT: no longer J16.6 (Pin_6), J23.6 (Pin_6), J27.6 (Pin_6)
- net /HOLD: no longer J16.5 (Pin_5), J23.5 (Pin_5), J27.5 (Pin_5)
- net /MEMIN: no longer J16.2 (Pin_2), J23.2 (Pin_2), J27.2 (Pin_2)
- net /RESET: no longer J16.8 (Pin_8), J23.8 (Pin_8), J27.8 (Pin_8)
- net /TAPE: now also J29.1 (Pin_1)
- net /WE: no longer J16.4 (Pin_4), J23.4 (Pin_4), J27.4 (Pin_4)
- new net AD1: J2.1 (Pin_1)
- new net AD10: J2.10 (Pin_10)
- new net AD11: J2.11 (Pin_11)
- new net AD12: J2.12 (Pin_12)
- new net AD13: J2.13 (Pin_13)
- new net AD14: J2.14 (Pin_14)
- new net AD15: J2.15 (Pin_15)
- new net AD2: J2.2 (Pin_2)
- new net AD3: J2.3 (Pin_3)
- new net AD4: J2.4 (Pin_4)
- new net AD5: J2.5 (Pin_5)
- new net AD6: J2.6 (Pin_6)
- new net AD7: J2.7 (Pin_7)
- new net AD8: J2.8 (Pin_8)
- new net AD9: J2.9 (Pin_9)
- new net DA0_2: D19.2 (A), J15.1 (Pin_1), U7.12 (RR1), U7.26 (TR1)
- new net DA0_3: D6.2 (A), J14.1 (Pin_1), J35.3 (Pin_3)
- new net DA1_2: D20.2 (A), J15.2 (Pin_2), U7.11 (RR2), U7.27 (TR2)
- new net DA1_3: J14.2 (Pin_2), J35.4 (Pin_4)
- new net DA2_2: J15.3 (Pin_3), U7.10 (RR3), U7.28 (TR3)
- new net DA2_3: J14.3 (Pin_3), J35.5 (Pin_5)
- new net DA3_2: J15.4 (Pin_4), U7.29 (TR4), U7.9 (RR4)
- new net DA3_3: J14.4 (Pin_4), J35.6 (Pin_6)
- new net DA4_2: J15.5 (Pin_5), U7.30 (TR5), U7.8 (RR5)
- new net DA4_3: J14.5 (Pin_5), J35.7 (Pin_7)
- new net DA5_2: J15.6 (Pin_6), U7.31 (TR6), U7.7 (RR6)
- new net DA5_3: J14.6 (Pin_6), J35.8 (Pin_8)
- new net DA6_2: J15.7 (Pin_7), U7.32 (TR7), U7.6 (RR7)
- new net DA6_3: J14.7 (Pin_7), J35.9 (Pin_9)
- new net DA7_2: J15.8 (Pin_8), U7.33 (TR8), U7.5 (RR8)
Other:
- moved on the sheet: J1, J10, J11, J12, J13, J14, J15, J16, J17, J18, J19, J2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

Commit message: 2026/4/6
Parts:
- added C25, C26: 1u, Capacitor_THT:C_Disc_D3.0mm_W1.6mm_P2.50mm, symbol Device:C
- added D7, D8: D, Diode_THT:D_DO-34_SOD68_P7.62mm_Horizontal, symbol Device:D
- added Q5, Q6: NPN, Package_TO_SOT_THT:TO-92_Inline_Wide, symbol Simulation_SPICE:NPN
- added R17, R20: 1k, Resistor_THT:R_Axial_DIN0207_L6.3mm_D2.5mm_P10.16mm_Horizontal, symbol Device:R
- added R18, R21: 10k, Resistor_THT:R_Axial_DIN0207_L6.3mm_D2.5mm_P10.16mm_Horizontal, symbol Device:R
- added R19, R27: 4.7k, Resistor_THT:R_Axial_DIN0207_L6.3mm_D2.5mm_P10.16mm_Horizontal, symbol Device:R
- R14: value 33k -> 220k
- R15: value 33k -> 4.7k
Connections:
- net DA8 is gone; now on net DA8_1: J3.9 (Pin_9)
- net DA9 is gone; now on net DA9_1: J3.10 (Pin_10)
- net +5V: now also R19.1, R27.1
- net GND: now also D7.2 (A), D8.2 (A), Q5.3 (E), Q6.3 (E), R17.1, R20.1
- net M0RERD: now also R18.1
- net M1RERD: now also R21.1
- net /PEN_M0: now also U12.1 (I4); no longer U12.2 (I5)
- net /PEN_M1: now also U12.13 (I3); no longer U12.1 (I4)
- net /TAPE: now also U12.2 (I5); no longer U12.3 (I6)
- net at U12.12 (I2): now also U14.2, U14.6
- net at U7.19 (DR), U8.9: now also C26.1; no longer U9.12
- net at U1.19 (DR), U6.9: now also C25.1; no longer U4.12
- net DA9_2: now reaches J15.10 (Pin_10)
- net DA9_2: now also D20.2 (A), U7.11 (RR2), U7.27 (TR2)
- net DA10_2: now reaches J15.11 (Pin_11)
- net DA10_2: now also U7.10 (RR3), U7.28 (TR3)
- net DA11_2: now reaches J15.12 (Pin_12)
- net DA11_2: now also U7.29 (TR4), U7.9 (RR4)
- net DA12_2: now reaches J15.13 (Pin_13)
- net DA12_2: now also U7.30 (TR5), U7.8 (RR5)
- net DA13_2: now reaches J15.14 (Pin_14)
- net DA13_2: now also U7.31 (TR6), U7.7 (RR6)
- net DA14_2: now reaches J15.15 (Pin_15)
- net DA14_2: now also U7.32 (TR7), U7.6 (RR7)
- net DA15_2: now reaches J15.16 (Pin_16)
- net DA15_2: now also U7.33 (TR8), U7.5 (RR8)
- net DA8_2: now reaches J15.9 (Pin_9)
- net DA8_2: now also D19.2 (A), U7.12 (RR1), U7.26 (TR1)
- net DA0_1 renamed DA8_1
- net DA8_1: no longer J3.1 (Pin_1)
- removed net DA0_2: D19.2 (A), J15.1 (Pin_1), U7.12 (RR1), U7.26 (TR1)
- net DA10 renamed DA10_1
- net DA10_1: now also U1.10 (RR3), U1.28 (TR3)
- net DA11 renamed DA11_1
- net DA11_1: now also U1.29 (TR4), U1.9 (RR4)
- net DA12 renamed DA12_1
- net DA12_1: now also U1.30 (TR5), U1.8 (RR5)
- net DA13 renamed DA13_1
- net DA13_1: now also U1.31 (TR6), U1.7 (RR6)
- net DA14 renamed DA14_1
- net DA14_1: now also U1.32 (TR7), U1.6 (RR7)
- net DA15 renamed DA15_1
- net DA15_1: now also U1.33 (TR8), U1.5 (RR8)
- net DA1_1 renamed DA9_1
- net DA9_1: no longer J3.2 (Pin_2)
- removed net DA1_2: D20.2 (A), J15.2 (Pin_2), U7.11 (RR2), U7.27 (TR2)
- removed net DA2_1: J3.3 (Pin_3), U1.10 (RR3), U1.28 (TR3)
- removed net DA2_2: J15.3 (Pin_3), U7.10 (RR3), U7.28 (TR3)
- removed net DA3_1: J3.4 (Pin_4), U1.29 (TR4), U1.9 (RR4)
- removed net DA3_2: J15.4 (Pin_4), U7.29 (TR4), U7.9 (RR4)
- removed net DA4_1: J3.5 (Pin_5), U1.30 (TR5), U1.8 (RR5)
- removed net DA4_2: J15.5 (Pin_5), U7.30 (TR5), U7.8 (RR5)
- removed net DA5_1: J3.6 (Pin_6), U1.31 (TR6), U1.7 (RR6)
- removed net DA5_2: J15.6 (Pin_6), U7.31 (TR6), U7.7 (RR6)
- removed net DA6_1: J3.7 (Pin_7), U1.32 (TR7), U1.6 (RR7)
- removed net DA6_2: J15.7 (Pin_7), U7.32 (TR7), U7.6 (RR7)
- removed net DA7_1: J3.8 (Pin_8), U1.33 (TR8), U1.5 (RR8)
- removed net DA7_2: J15.8 (Pin_8), U7.33 (TR8), U7.5 (RR8)
- net /M0IQR: no longer names the net of U1.18 (DRR)
- net /M0IQR: now also Q5.1 (C), R19.2
- net /M1IQR: no longer names the net of U7.18 (DRR)
- net /M1IQR: now also Q6.1 (C), R27.2
- new net: C25.2, D7.1 (K), R17.2, U4.12
- new net: Q5.2 (B), R18.2
- new net: C26.2, D8.1 (K), R20.2, U9.12
- new net: Q6.2 (B), R21.2
- new net DA0: J3.1 (Pin_1)
- new net DA1: J3.2 (Pin_2)
- new net DA2: J3.3 (Pin_3)
- new net DA3: J3.4 (Pin_4)
- new net DA4: J3.5 (Pin_5)
- new net DA5: J3.6 (Pin_6)
- new net DA6: J3.7 (Pin_7)
- new net DA7: J3.8 (Pin_8)
Other:
- moved on the sheet: J15, J16, J17, J18, J19, U4D, U6B, U6D, U8B, U8D, U9D

Commit message: 2026/4/7
Parts:
- added J31, J33, J36, J37: Conn_01x14_Pin, Connector_PinHeader_2.54mm:PinHeader_1x14_P2.54mm_Vertical, symbol Connector:Conn_01x14_Pin
Connections:
- net DA9_3: now reaches J14.10 (Pin_10)
- net DA9_3: now also J35.4 (Pin_4)
- net DA10_3: now reaches J14.11 (Pin_11)
- net DA10_3: now also J35.5 (Pin_5)
- net DA11_3: now reaches J14.12 (Pin_12)
- net DA11_3: now also J35.6 (Pin_6)
- net DA12_3: now reaches J14.13 (Pin_13)
- net DA12_3: now also J35.7 (Pin_7)
- net DA13_3: now reaches J14.14 (Pin_14)
- net DA13_3: now also J35.8 (Pin_8)
- net DA14_3: now reaches J14.15 (Pin_15)
- net DA14_3: now also J35.9 (Pin_9)
- net DA8_3: now reaches J14.9 (Pin_9)
- net DA8_3: now also D6.2 (A), J35.3 (Pin_3)
- removed net DA0_3: D6.2 (A), J14.1 (Pin_1), J35.3 (Pin_3)
- net DA1_3: no longer names the net of J14.2 (Pin_2)
- net DA1_3: no longer J35.4 (Pin_4)
- net DA2_3: no longer names the net of J14.3 (Pin_3)
- net DA2_3: no longer J35.5 (Pin_5)
- net DA3_3: no longer names the net of J14.4 (Pin_4)
- net DA3_3: no longer J35.6 (Pin_6)
- net DA4_3: no longer names the net of J14.5 (Pin_5)
- net DA4_3: no longer J35.7 (Pin_7)
- net DA5_3: no longer names the net of J14.6 (Pin_6)
- net DA5_3: no longer J35.8 (Pin_8)
- net DA6_3: no longer names the net of J14.7 (Pin_7)
- net DA6_3: no longer J35.9 (Pin_9)
- new net: J31.1 (Pin_1), J33.1 (Pin_1), J36.1 (Pin_1), J37.1 (Pin_1)
- new net: J31.10 (Pin_10), J33.10 (Pin_10), J36.10 (Pin_10), J37.10 (Pin_10)
- new net: J31.11 (Pin_11), J33.11 (Pin_11), J36.11 (Pin_11), J37.11 (Pin_11)
- new net: J31.12 (Pin_12), J33.12 (Pin_12), J36.12 (Pin_12), J37.12 (Pin_12)
- new net: J31.13 (Pin_13), J33.13 (Pin_13), J36.13 (Pin_13), J37.13 (Pin_13)
- new net: J31.14 (Pin_14), J33.14 (Pin_14), J36.14 (Pin_14), J37.14 (Pin_14)
- new net: J31.2 (Pin_2), J33.2 (Pin_2), J36.2 (Pin_2), J37.2 (Pin_2)
- new net: J31.3 (Pin_3), J33.3 (Pin_3), J36.3 (Pin_3), J37.3 (Pin_3)
- new net: J31.4 (Pin_4), J33.4 (Pin_4), J36.4 (Pin_4), J37.4 (Pin_4)
- new net: J31.5 (Pin_5), J33.5 (Pin_5), J36.5 (Pin_5), J37.5 (Pin_5)
- new net: J31.6 (Pin_6), J33.6 (Pin_6), J36.6 (Pin_6), J37.6 (Pin_6)
- new net: J31.7 (Pin_7), J33.7 (Pin_7), J36.7 (Pin_7), J37.7 (Pin_7)
- new net: J31.8 (Pin_8), J33.8 (Pin_8), J36.8 (Pin_8), J37.8 (Pin_8)
- new net: J31.9 (Pin_9), J33.9 (Pin_9), J36.9 (Pin_9), J37.9 (Pin_9)

Commit message: 2026/4/9
Parts:
- C4: value 470nF -> 47nF
Changed lines of the file:
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@@
 			)
 		)
-		(property "Value" "470nF"
+		(property "Value" "47nF"
 			(at 300.736 271.526 0)
 			(effects

Commit message: 2026/6/10
Parts:
- removed D11, D12: D_Schottky, Diode_THT:D_DO-34_SOD68_P7.62mm_Horizontal, symbol Device:D_Schottky
- added Q7, Q8: NPN, Package_TO_SOT_THT:TO-92_Inline_Wide, symbol Simulation_SPICE:NPN
- added R28, R29: 10k, Resistor_THT:R_Axial_DIN0207_L6.3mm_D2.5mm_P10.16mm_Horizontal, symbol Device:R
Connections:
- net +5V: now also Q7.1 (C), Q8.1 (C)
- net at R8.2, U11.4 (E1), U13.4 (E1): now also Q7.3 (E), Q8.3 (E)
- net at U3.3: now also R29.2
- net at U3.6: now also R28.2
- new net: Q8.2 (B), R29.1
- new net: Q7.2 (B), R28.1
